File: proteus125honda.kicad_pcb (KiCad board)
At the start: 2 copper layers, 153 x 151.3 mm, 4 parts, among them J1 1318612-1, J2 Conn_01x35, J3 Conn_01x35, J4 Conn_01x23

Commit message: Upd pinout
Parts:
- added D1: D_Schottky, Diode_SMD:D_SMA, F.Cu at (296.0, 159.8)
- added F1: Fuse-Pad-Pad, hellen-one-common:PAD-1206-PAD, F.Cu at (366.2, 108.4)
- added F2: Fuse-Pad-Pad, hellen-one-common:PAD-1206-PAD, F.Cu at (287.8, 159.2)
- added J5: Conn_01x35, lib:ampseal-35-2, F.Cu at (222.0, 146.8)
- added J6: Conn_01x23, lib:ampseal-23, F.Cu at (171.0, 168.8)
- added M1: Module-wbo-0.2, hellen-one-wbo-0.2:wbo, F.Cu at (329.4, 63.2)
- added M2: Module-can-0.1, hellen-one-can-0.1:can, F.Cu at (320.6, 48.2)
- added P1: Pad, hellen-one-common:PAD-TH, F.Cu at (351.7, 137.9)
- added P10: Pad, hellen-one-common:PAD-TH, F.Cu at (313.3, 159.4)
- added P11: Pad, hellen-one-common:PAD-TH, F.Cu at (390.5, 112.3)
- added P12: Pad, hellen-one-common:PAD-TH, F.Cu at (371.6, 112.3)
- added P13: Pad, hellen-one-common:PAD-TH, F.Cu at (371.9, 123.7)
- added P14: Pad, hellen-one-common:PAD-TH, F.Cu at (371.9, 119.9)
- added P15: Pad, hellen-one-common:PAD-TH, F.Cu at (408.4, 92.2)
- added P16: Pad, hellen-one-common:PAD-TH, F.Cu at (289.4, 162.8)
- added P17: Pad, hellen-one-common:PAD-TH, F.Cu at (351.7, 149.3)
- added P18: Pad, hellen-one-common:PAD-TH, F.Cu at (375.3, 116.1)
- added P19: Pad, hellen-one-common:PAD-TH, F.Cu at (383.6, 108.6)
- added P2: Pad, hellen-one-common:PAD-TH, F.Cu at (320.8, 159.4)
- added P20: Pad, hellen-one-common:PAD-TH, F.Cu at (355.5, 134.1)
- added P21: Pad, hellen-one-common:PAD-TH, F.Cu at (332.2, 159.4)
- added P22: Pad, hellen-one-common:PAD-TH, F.Cu at (175.0, 94.8)
- added P23: Pad, hellen-one-common:PAD-TH, F.Cu at (364.0, 115.7)
- added P24: Pad, hellen-one-common:PAD-TH, F.Cu at (355.5, 141.7)
- added P25: Pad, hellen-one-common:PAD-TH, F.Cu at (382.9, 116.1)
- added P26: Pad, hellen-one-common:PAD-TH, F.Cu at (366.8, 138.4)
- added P27: Pad, hellen-one-common:PAD-TH, F.Cu at (368.1, 123.3)
- added P28: Pad, hellen-one-common:PAD-TH, F.Cu at (359.2, 144.7)
- added P29: Pad, hellen-one-common:PAD-TH, F.Cu at (347.9, 145.5)
- added P3: Pad, hellen-one-common:PAD-TH, F.Cu at (379.1, 112.3)
- added P30: Pad, hellen-one-common:PAD-TH, F.Cu at (404.6, 99.8)
- added P31: Pad, hellen-one-common:PAD-TH, F.Cu at (363.0, 138.4)
- added P32: Pad, hellen-one-common:PAD-TH, F.Cu at (404.6, 92.2)
- added P33: Pad, hellen-one-common:PAD-TH, F.Cu at (376.0, 108.6)
- added P34: Pad, hellen-one-common:PAD-TH, F.Cu at (309.5, 159.4)
- added P35: Pad, hellen-one-common:PAD-TH, F.Cu at (371.9, 131.2)
- added P36: Pad, hellen-one-common:PAD-TH, F.Cu at (375.3, 112.3)
- added P37: Pad, hellen-one-common:PAD-TH, F.Cu at (379.4, 119.9)
- added P38: Pad, hellen-one-common:PAD-TH, F.Cu at (379.8, 108.6)
- added P39: Pad, hellen-one-common:PAD-TH, F.Cu at (372.3, 108.6)
- added P4: Pad, hellen-one-common:PAD-TH, F.Cu at (347.9, 149.3)
- added P40: Pad, hellen-one-common:PAD-TH, F.Cu at (368.1, 130.8)
- added P41: Pad, hellen-one-common:PAD-TH, F.Cu at (367.8, 115.7)
- added P42: Pad, hellen-one-common:PAD-TH, F.Cu at (359.2, 148.5)
- added P43: Pad, hellen-one-common:PAD-TH, F.Cu at (317.0, 159.4)
- added P44: Pad, hellen-one-common:PAD-TH, F.Cu at (351.7, 145.5)
- added P45: Pad, hellen-one-common:PAD-TH, F.Cu at (379.4, 123.7)
- added P46: Pad, hellen-one-common:PAD-TH, F.Cu at (394.9, 108.6)
- added P47: Pad, hellen-one-common:PAD-TH, F.Cu at (364.0, 119.5)
- added P48: Pad, hellen-one-common:PAD-TH, F.Cu at (408.4, 96.0)
- added P49: Pad, hellen-one-common:PAD-TH, F.Cu at (364.0, 111.9)
- added P5: Pad, hellen-one-common:PAD-TH, F.Cu at (364.3, 123.3)
- added P50: Pad, hellen-one-common:PAD-TH, F.Cu at (360.5, 125.8)
- added P51: Pad, hellen-one-common:PAD-TH, F.Cu at (375.6, 127.5)
- added P52: Pad, hellen-one-common:PAD-TH, F.Cu at (347.9, 153.0)
- added P53: Pad, hellen-one-common:PAD-TH, F.Cu at (355.5, 145.5)
- added P54: Pad, hellen-one-common:PAD-TH, F.Cu at (383.2, 119.9)
- added P55: Pad, hellen-one-common:PAD-TH, F.Cu at (301.9, 159.4)
- added P56: Pad, hellen-one-common:PAD-TH, F.Cu at (364.3, 130.8)
- added P57: Pad, hellen-one-common:PAD-TH, F.Cu at (379.1, 116.1)
- added P58: Pad, hellen-one-common:PAD-TH, F.Cu at (351.7, 141.7)
- added P59: Pad, hellen-one-common:PAD-TH, F.Cu at (368.1, 134.6)
- added P6: Pad, hellen-one-common:PAD-TH, F.Cu at (387.4, 108.6)
- added P60: Pad, hellen-one-common:PAD-TH, F.Cu at (382.9, 112.3)
- added P61: Pad, hellen-one-common:PAD-TH, F.Cu at (343.5, 159.4)
- added P62: Pad, hellen-one-common:PAD-TH, F.Cu at (355.5, 137.9)
- added P63: Pad, hellen-one-common:PAD-TH, F.Cu at (371.9, 127.5)
- added P64: Pad, hellen-one-common:PAD-TH, F.Cu at (368.1, 127.0)
- added P65: Pad, hellen-one-common:PAD-TH, F.Cu at (386.7, 112.3)
- added P66: Pad, hellen-one-common:PAD-TH, F.Cu at (363.0, 142.2)
- added P67: Pad, hellen-one-common:PAD-TH, F.Cu at (347.9, 137.9)
- added P68: Pad, hellen-one-common:PAD-TH, F.Cu at (359.2, 140.9)
- added P69: Pad, hellen-one-common:PAD-TH, F.Cu at (375.6, 119.9)
- added P7: Pad, hellen-one-common:PAD-TH, F.Cu at (305.7, 159.4)
- added P70: Pad, hellen-one-common:PAD-TH, F.Cu at (412.2, 92.2)
- added P71: Pad, hellen-one-common:PAD-TH, F.Cu at (324.6, 159.4)
- added P72: Pad, hellen-one-common:PAD-TH, F.Cu at (367.8, 111.9)
- added P73: Pad, hellen-one-common:PAD-TH, F.Cu at (339.7, 159.4)
- added P74: Pad, hellen-one-common:PAD-TH, F.Cu at (367.8, 119.5)
- added P75: Pad, hellen-one-common:PAD-TH, F.Cu at (347.9, 134.1)
- added P76: Pad, hellen-one-common:PAD-TH, F.Cu at (359.2, 137.2)
- added P77: Pad, hellen-one-common:PAD-TH, F.Cu at (391.2, 108.6)
- added P78: Pad, hellen-one-common:PAD-TH, F.Cu at (404.6, 103.6)
- added P79: Pad, hellen-one-common:PAD-TH, F.Cu at (404.6, 96.0)
- added P8: Pad, hellen-one-common:PAD-TH, F.Cu at (360.5, 133.4)
- added P80: Pad, hellen-one-common:PAD-TH, F.Cu at (328.4, 159.4)
- added P81: Pad, hellen-one-common:PAD-TH, F.Cu at (351.7, 134.1)
- added P82: Pad, hellen-one-common:PAD-TH, F.Cu at (360.5, 129.6)
- added P83: Pad, hellen-one-common:PAD-TH, F.Cu at (347.9, 141.7)
- added P84: Pad, hellen-one-common:PAD-TH, F.Cu at (335.9, 159.4)
- added P85: Pad, hellen-one-common:PAD-TH, F.Cu at (364.3, 134.6)
- added P86: Pad, hellen-one-common:PAD-TH, F.Cu at (371.6, 116.1)
- added P87: Pad, hellen-one-common:PAD-TH, F.Cu at (375.6, 123.7)
- added P88: Pad, hellen-one-common:PAD-TH, F.Cu at (364.3, 127.0)
- added P9: Pad, hellen-one-common:PAD-TH, F.Cu at (386.7, 116.1)
- J2: value Conn_01x35 -> XH-8A; footprint lib:ampseal-35 -> hellen-one-common:XH-8A
- J3: value Conn_01x35 -> Conn_01x06; footprint lib:ampseal-35-2 -> Connector_PinHeader_2.54mm:PinHeader_1x06_P2.54mm_Vertical
- J4: value Conn_01x23 -> Conn_01x35; footprint lib:ampseal-23 -> lib:ampseal-35
- moved J2 267.9 mm to (374.0, 57.8)
- moved J3 142.4 mm to (343.6, 66.8), turned to -90 degrees
- moved J4 52.5 mm to (121.0, 146.8), turned to -90 degrees
Connections:
- J1 pad A1: (no net) -> /IN_KNOCK
- J1 pad A10: (no net) -> Net-(J1-PadA10)
- J1 pad A11: (no net) -> /LS14
- J1 pad A12: (no net) -> /LS13
- J1 pad A13: (no net) -> /IGN4
- J1 pad A14: (no net) -> /IGN3
- J1 pad A15: (no net) -> /IGN2
- J1 pad A16: (no net) -> /IGN1
- J1 pad A18: (no net) -> /DIGITAL_3
- J1 pad A19: (no net) -> /DIGITAL_4
- J1 pad A2: (no net) -> Net-(F1-Pad1)
- J1 pad A20: (no net) -> /5V_SENSOR_1
- J1 pad A21: (no net) -> /5V_SENSOR_1
- J1 pad A23: (no net) -> GND
- J1 pad A24: (no net) -> GND
- J1 pad A25: (no net) -> /AV1
- J1 pad A26: (no net) -> /AV2
- J1 pad A28: (no net) -> Net-(J1-PadA28)
- J1 pad A29: (no net) -> /AV3
- J1 pad A3: (no net) -> Net-(F2-Pad1)
- J1 pad A30: (no net) -> /IN_MAP
- J1 pad A31: (no net) -> Net-(J1-PadA31)
- J1 pad A4: (no net) -> GND
- J1 pad A5: (no net) -> GND
- J1 pad A6: (no net) -> /DIGITAL_1
- J1 pad A7: (no net) -> /DIGITAL_2
- J1 pad A8: (no net) -> GND
- J1 pad A9: (no net) -> GND
- J1 pad B1: (no net) -> /LS15
- J1 pad B10: (no net) -> Net-(J1-PadB10)
- J1 pad B11: (no net) -> /DIGITAL_5
- J1 pad B13: (no net) -> Net-(J1-PadB13)
- J1 pad B15: (no net) -> /OUT_MCS
- J1 pad B17: (no net) -> /AT1
- J1 pad B18: (no net) -> Net-(J1-PadB18)
- J1 pad B19: (no net) -> Net-(J1-PadB19)
- J1 pad B2: (no net) -> /LS1
- J1 pad B20: (no net) -> Net-(J1-PadB20)
- J1 pad B21: (no net) -> /OUT_PURGE
- J1 pad B22: (no net) -> /AV4
- J1 pad B3: (no net) -> /LS2
- J1 pad B4: (no net) -> /LS3
- J1 pad B5: (no net) -> /LS4
- J1 pad B6: (no net) -> /LS16
- J1 pad B8: (no net) -> /AT2
- J1 pad C1: (no net) -> Net-(J1-PadC1)
- J1 pad C10: (no net) -> Net-(J1-PadC10)
- J1 pad C11: (no net) -> Net-(J1-PadC11)
- J1 pad C12: (no net) -> Net-(J1-PadC12)
- J1 pad C13: (no net) -> Net-(J1-PadC13)
- J1 pad C14: (no net) -> Net-(J1-PadC14)
- J1 pad C15: (no net) -> Net-(J1-PadC15)
- J1 pad C16: (no net) -> Net-(J1-PadC16)
- J1 pad C17: (no net) -> Net-(J1-PadC17)
- J1 pad C18: (no net) -> Net-(J1-PadC18)
- J1 pad C19: (no net) -> Net-(J1-PadC19)
- J1 pad C2: (no net) -> Net-(J1-PadC2)
- J1 pad C20: (no net) -> Net-(J1-PadC20)
- J1 pad C21: (no net) -> Net-(J1-PadC21)
- J1 pad C22: (no net) -> Net-(J1-PadC22)
- J1 pad C3: (no net) -> Net-(J1-PadC3)
- J1 pad C4: (no net) -> Net-(J1-PadC4)
- J1 pad C5: (no net) -> Net-(J1-PadC5)
- J1 pad C6: (no net) -> Net-(J1-PadC6)
- J1 pad C7: (no net) -> Net-(J1-PadC7)
- J1 pad C8: (no net) -> Net-(J1-PadC8)
- J1 pad C9: (no net) -> Net-(J1-PadC9)
- J1 pad D10: (no net) -> Net-(J1-PadD10)
- J1 pad D12: (no net) -> Net-(J1-PadD12)
- J1 pad D15: (no net) -> Net-(J1-PadD15)
- J1 pad D2: (no net) -> Net-(J1-PadD2)
- J1 pad D3: (no net) -> Net-(J1-PadD3)
- J1 pad D5: (no net) -> Net-(J1-PadD5)
- J1 pad D6: (no net) -> Net-(J1-PadD6)
- J1 pad D8: (no net) -> Net-(J1-PadD8)
- J1 pad D9: (no net) -> Net-(J1-PadD9)
- J1 pad E1: (no net) -> Net-(J1-PadE1)
- J1 pad E11: (no net) -> /CAN+
- J1 pad E12: (no net) -> Net-(J1-PadE12)
- J1 pad E13: (no net) -> Net-(J1-PadE13)
- J1 pad E14: (no net) -> /AV6
- J1 pad E15: (no net) -> Net-(J1-PadE15)
- J1 pad E16: (no net) -> Net-(J1-PadE16)
- J1 pad E17: (no net) -> /OUT_FUEL_PUMP
- J1 pad E18: (no net) -> Net-(J1-PadE18)
- J1 pad E19: (no net) -> /OUT_VENT
- J1 pad E2: (no net) -> Net-(J1-PadE2)
- J1 pad E20: (no net) -> Net-(J1-PadE20)
- J1 pad E21: (no net) -> Net-(J1-PadE21)
- J1 pad E22: (no net) -> /AV5
- J1 pad E23: (no net) -> Net-(J1-PadE23)
- J1 pad E24: (no net) -> /CAN-
- J1 pad E25: (no net) -> Net-(J1-PadE25)
- J1 pad E26: (no net) -> Net-(J1-PadE26)
- J1 pad E27: (no net) -> Net-(J1-PadE27)
- J1 pad E29: (no net) -> Net-(J1-PadE29)
- J1 pad E3: (no net) -> Net-(J1-PadE3)
- J1 pad E30: (no net) -> Net-(J1-PadE30)
- J1 pad E31: (no net) -> /LS6
- J1 pad E4: (no net) -> GND
- J1 pad E5: (no net) -> /5V_SENSOR_1
- J1 pad E7: (no net) -> /LS5
- J1 pad E8: (no net) -> /OUT_MAF_RELAY
- J1 pad E9: (no net) -> /12V_RAW
- J2 pad 1: (no net) -> GND
- J2 pad 2: (no net) -> GND
- J2 pad 3: (no net) -> /WBO_H-
- J2 pad 4: (no net) -> /WBO_H-
- J2 pad 5: (no net) -> /WBO_R_Trim
- J2 pad 6: (no net) -> /WBO_Ip
- J2 pad 7: (no net) -> /WBO_Vs/Ip
- J2 pad 8: (no net) -> /WBO_Vs
- J3 pad 1: GND -> Net-(J3-Pad1)
- J3 pad 2: GND -> Net-(J3-Pad2)
- J3 pad 4: GND -> Net-(J3-Pad4)
- J3 pad 5: GND -> Net-(J3-Pad5)
- J3 pad 6: GND -> (no net)
- J4 pad 1: (no net) -> /HS2
- J4 pad 10: (no net) -> /LS13
- J4 pad 11: (no net) -> /LS14
- J4 pad 12: (no net) -> /LS15
- J4 pad 13: (no net) -> /HS3
- J4 pad 14: GND -> /HS4
- J4 pad 15: (no net) -> /LS2
- J4 pad 16: (no net) -> /LS4
- J4 pad 17: (no net) -> GND
- J4 pad 18: (no net) -> GND
- J4 pad 19: GND -> /OUT_PURGE
- J4 pad 2: (no net) -> /HS1
- J4 pad 20: GND -> /OUT_VENT
- J4 pad 22: (no net) -> /IGN3
- J4 pad 23: (no net) -> /LS16
- J4 pad 3: (no net) -> /LS1
- J4 pad 4: (no net) -> /LS3
- J4 pad 5: (no net) -> /LS5
- J4 pad 6: (no net) -> /LS6
- J4 pad 7: (no net) -> /OUT_MAF_RELAY
- J4 pad 8: (no net) -> /OUT_FUEL_PUMP
- J4 pad 9: (no net) -> /LS11

Commit message: Upd pcb
Parts:
- added J10: Conn_01x01, MountingHole:MountingHole_4.5mm, F.Cu at (171.5, 213.8)
- added J11: Conn_01x01, MountingHole:MountingHole_4.5mm, F.Cu at (243.9, 93.0)
- added J12: Conn_01x01, MountingHole:MountingHole_4.5mm, F.Cu at (243.9, 201.0)
- added J13: Conn_01x01, MountingHole:MountingHole_4.5mm, F.Cu at (99.0, 201.0)
- added J7: Conn_01x01, MountingHole:MountingHole_4.5mm, F.Cu at (99.0, 138.0)
- added J8: Conn_01x01, MountingHole:MountingHole_4.5mm, F.Cu at (243.9, 153.5)
- added J9: Conn_01x01, MountingHole:MountingHole_4.5mm, F.Cu at (99.0, 93.0)
- added P89: Pad, hellen-one-common:PAD-TH, F.Cu at (195.5, 93.8)
- added P90: Pad, hellen-one-common:PAD-TH, F.Cu at (132.0, 93.8)
- added P91: Pad, hellen-one-common:PAD-TH, F.Cu at (117.0, 102.8)
- added P92: Pad, hellen-one-common:PAD-TH, F.Cu at (129.0, 98.3)
- added P93: Pad, hellen-one-common:PAD-TH, F.Cu at (201.0, 142.8)
- added P94: Pad, hellen-one-common:PAD-TH, F.Cu at (201.0, 145.9)
- added P95: Pad, hellen-one-common:PAD-TH, F.Cu at (201.0, 139.1)
- added P96: Pad, hellen-one-common:PAD-TH, F.Cu at (204.0, 129.4)
- added P97: Pad, hellen-one-common:PAD-TH, F.Cu at (136.0, 133.3)
- moved P48 276.4 mm to (132.0, 98.4)
- moved P46 272.3 mm to (123.0, 93.8)
- moved P51 263.3 mm to (114.0, 98.3)
- moved P40 262.7 mm to (108.0, 93.8)
- moved P45 261.1 mm to (120.0, 93.8)
- moved P41 260.4 mm to (108.0, 98.3)
- moved P32 260.1 mm to (144.5, 93.8)
- moved P77 257.4 mm to (136.0, 142.3)
- moved P54 255.5 mm to (129.0, 93.8)
- moved P50 253.6 mm to (108.0, 102.8)
- moved P60 250.4 mm to (136.0, 154.3), turned to -90 degrees
- moved P42 248.3 mm to (117.0, 93.8)
- moved P57 246.6 mm to (136.0, 157.3), turned to -90 degrees
- moved P44 243.2 mm to (114.0, 93.8)
- moved P78 241.2 mm to (168.0, 150.3)
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Connections:
- net /IN_MAP renamed /AV7
- net /OUT_FUEL_PUMP renamed /LS9
- J1 pad B21: /OUT_PURGE -> Net-(J1-PadB21)
- J1 pad E14: /AV6 -> Net-(J1-PadE14)
- J1 pad E19: /OUT_VENT -> Net-(J1-PadE19)
- J1 pad E8: /OUT_MAF_RELAY -> Net-(J1-PadE8)
- J4 pad 19: /OUT_PURGE -> /LS8
- J4 pad 20: /OUT_VENT -> /LS10
- J4 pad 21: (no net) -> /LS12
- J4 pad 7: /OUT_MAF_RELAY -> /LS7
Routing:
- net /5V_SENSOR_1: track 0.00 -> 245.3 mm, vias 0 -> 2
- net /DIGITAL_3: track 0.00 -> 181.2 mm, vias 0 -> 1
- net /DIGITAL_2: track 0.00 -> 179.3 mm, vias 0 -> 1
- net /AV7: track 0.00 -> 177.3 mm, vias 0 -> 1
- net /DIGITAL_4: track 0.00 -> 173.3 mm, vias 0 -> 1
- net /DIGITAL_1: track 0.00 -> 170.1 mm, vias 0 -> 1
- net /AV3: track 0.00 -> 167.7 mm, vias 0 -> 1
- net /IN_KNOCK: track 0.00 -> 163.6 mm, vias 0 -> 2
- net /LS5: track 0.00 -> 155.5 mm, vias 0 -> 3
- net /LS9: track 0.00 -> 154.8 mm, vias 0 -> 3
- net /LS6: track 0.00 -> 152.0 mm, vias 0 -> 2
- net /CAN+: track 0.00 -> 148.3 mm
- net /AV1: track 0.00 -> 147.3 mm, vias 0 -> 1
- net /AV2: track 0.00 -> 146.7 mm, vias 0 -> 1
- net /CAN-: track 0.00 -> 139.3 mm, vias 0 -> 2
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- added copper zone on B.Cu, net GND
- added copper zone on F.Cu, net GND
Other:
- outline, holes or cut-outs redrawn

Commit message: Proteus-compatible component
Parts:
- removed J4: Conn_01x35, lib:ampseal-35
- removed J5: Conn_01x35, lib:ampseal-35-2
- removed J6: Conn_01x23, lib:ampseal-23
- added D2: proteus, kicad6-libraries:proteus, F.Cu at (238.5, 119.0)
- added G***: LOGO, LOGO, F.Cu at (124.0, 201.8)
- added G1: PROTO_AREA, hellen-one-common:PROTO_AREA, F.Cu at (285.4, 122.2)
- added G2: PROTO_AREA, hellen-one-common:PROTO_AREA, F.Cu at (272.1, 114.0)
- added G3: PROTO_AREA, hellen-one-common:PROTO_AREA, F.Cu at (285.4, 114.0)
- added G4: PROTO_AREA, hellen-one-common:PROTO_AREA, F.Cu at (272.1, 130.4)
- added G5: PROTO_AREA, hellen-one-common:PROTO_AREA, F.Cu at (272.1, 122.2)
- J1: footprint lib:13186121 -> kicad6-libraries:TE_1318612-1
- moved P56 194.3 mm to (329.3, 170.7)
- moved P57 194.3 mm to (329.3, 176.7)
- moved P58 194.3 mm to (329.3, 179.7)
- moved P59 194.3 mm to (329.3, 187.7)
- moved P60 194.3 mm to (329.3, 173.7)
- moved P74 194.3 mm to (329.3, 164.7)
- moved P75 194.3 mm to (329.3, 167.7)
- moved P76 194.3 mm to (329.3, 157.2)
- moved P77 194.3 mm to (329.3, 161.7)
- moved P97 194.3 mm to (329.3, 152.7)
- moved P61 117.4 mm to (319.7, 192.6)
- moved P62 117.4 mm to (319.7, 183.6)
- moved P63 117.4 mm to (319.7, 158.0)
- moved P64 117.4 mm to (319.7, 189.6)
- moved P65 117.4 mm to (319.7, 180.6)
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Connections:
- J1 pad A10: Net-(J1-PadA10) -> Net-(P1-Pad1)
- J1 pad A17: (no net) -> unconnected-(J1-PadA17)
- J1 pad A22: (no net) -> unconnected-(J1-PadA22)
- J1 pad A27: (no net) -> unconnected-(J1-PadA27)
- J1 pad A28: Net-(J1-PadA28) -> Net-(P2-Pad1)
- J1 pad A31: Net-(J1-PadA31) -> Net-(P3-Pad1)
- J1 pad B10: Net-(J1-PadB10) -> Net-(P4-Pad1)
- J1 pad B12: (no net) -> unconnected-(J1-PadB12)
- J1 pad B13: Net-(J1-PadB13) -> Net-(P5-Pad1)
- J1 pad B14: (no net) -> unconnected-(J1-PadB14)
- J1 pad B16: (no net) -> unconnected-(J1-PadB16)
- J1 pad B18: Net-(J1-PadB18) -> Net-(P6-Pad1)
- J1 pad B19: Net-(J1-PadB19) -> Net-(P7-Pad1)
- J1 pad B20: Net-(J1-PadB20) -> Net-(P8-Pad1)
- J1 pad B21: Net-(J1-PadB21) -> Net-(P89-Pad1)
- J1 pad B23: (no net) -> unconnected-(J1-PadB23)
- J1 pad B24: (no net) -> unconnected-(J1-PadB24)
- J1 pad B7: (no net) -> unconnected-(J1-PadB7)
- J1 pad B9: (no net) -> unconnected-(J1-PadB9)
- J1 pad C1: Net-(J1-PadC1) -> Net-(P9-Pad1)
- J1 pad C10: Net-(J1-PadC10) -> Net-(P18-Pad1)
- J1 pad C11: Net-(J1-PadC11) -> Net-(P19-Pad1)
- J1 pad C12: Net-(J1-PadC12) -> Net-(P20-Pad1)
- J1 pad C13: Net-(J1-PadC13) -> Net-(P21-Pad1)
- J1 pad C14: Net-(J1-PadC14) -> Net-(P22-Pad1)
- J1 pad C15: Net-(J1-PadC15) -> Net-(P23-Pad1)
- J1 pad C16: Net-(J1-PadC16) -> Net-(P24-Pad1)
- J1 pad C17: Net-(J1-PadC17) -> Net-(P25-Pad1)
- J1 pad C18: Net-(J1-PadC18) -> Net-(P26-Pad1)
- J1 pad C19: Net-(J1-PadC19) -> Net-(P27-Pad1)
- J1 pad C2: Net-(J1-PadC2) -> Net-(P10-Pad1)
- J1 pad C20: Net-(J1-PadC20) -> Net-(P28-Pad1)
- J1 pad C21: Net-(J1-PadC21) -> Net-(P29-Pad1)
- J1 pad C22: Net-(J1-PadC22) -> Net-(P30-Pad1)
- J1 pad C3: Net-(J1-PadC3) -> Net-(P11-Pad1)
- J1 pad C4: Net-(J1-PadC4) -> Net-(P12-Pad1)
- J1 pad C5: Net-(J1-PadC5) -> Net-(P13-Pad1)
- J1 pad C6: Net-(J1-PadC6) -> Net-(P14-Pad1)
- J1 pad C7: Net-(J1-PadC7) -> Net-(P15-Pad1)
- J1 pad C8: Net-(J1-PadC8) -> Net-(P16-Pad1)
- J1 pad C9: Net-(J1-PadC9) -> Net-(P17-Pad1)
- J1 pad D1: (no net) -> unconnected-(J1-PadD1)
- J1 pad D10: Net-(J1-PadD10) -> Net-(P37-Pad1)
- J1 pad D11: (no net) -> unconnected-(J1-PadD11)
- J1 pad D12: Net-(J1-PadD12) -> Net-(P38-Pad1)
- J1 pad D13: (no net) -> unconnected-(J1-PadD13)
- J1 pad D14: (no net) -> unconnected-(J1-PadD14)
- J1 pad D15: Net-(J1-PadD15) -> Net-(P39-Pad1)
- J1 pad D16: (no net) -> unconnected-(J1-PadD16)
- J1 pad D17: (no net) -> unconnected-(J1-PadD17)
- J1 pad D2: Net-(J1-PadD2) -> Net-(P31-Pad1)
- J1 pad D3: Net-(J1-PadD3) -> Net-(P32-Pad1)
- J1 pad D4: (no net) -> unconnected-(J1-PadD4)
- J1 pad D5: Net-(J1-PadD5) -> Net-(P33-Pad1)
- J1 pad D6: Net-(J1-PadD6) -> Net-(P34-Pad1)
- J1 pad D7: (no net) -> unconnected-(J1-PadD7)
- J1 pad D8: Net-(J1-PadD8) -> Net-(P35-Pad1)
- J1 pad D9: Net-(J1-PadD9) -> Net-(P36-Pad1)
- J1 pad E1: Net-(J1-PadE1) -> Net-(P40-Pad1)
- J1 pad E10: (no net) -> unconnected-(J1-PadE10)
- J1 pad E12: Net-(J1-PadE12) -> Net-(P43-Pad1)
- J1 pad E13: Net-(J1-PadE13) -> Net-(P44-Pad1)
- J1 pad E14: Net-(J1-PadE14) -> Net-(P91-Pad1)
- J1 pad E15: Net-(J1-PadE15) -> Net-(P45-Pad1)
- J1 pad E16: Net-(J1-PadE16) -> Net-(P46-Pad1)
- J1 pad E18: Net-(J1-PadE18) -> Net-(P47-Pad1)
- J1 pad E19: Net-(J1-PadE19) -> Net-(P92-Pad1)
- J1 pad E2: Net-(J1-PadE2) -> Net-(P41-Pad1)
- J1 pad E20: Net-(J1-PadE20) -> Net-(P48-Pad1)
- J1 pad E21: Net-(J1-PadE21) -> Net-(P49-Pad1)
- J1 pad E23: Net-(J1-PadE23) -> Net-(P50-Pad1)
- J1 pad E25: Net-(J1-PadE25) -> Net-(P51-Pad1)
- J1 pad E26: Net-(J1-PadE26) -> Net-(P52-Pad1)
- J1 pad E27: Net-(J1-PadE27) -> Net-(P53-Pad1)
- J1 pad E28: (no net) -> unconnected-(J1-PadE28)
- J1 pad E29: Net-(J1-PadE29) -> Net-(P54-Pad1)
- J1 pad E3: Net-(J1-PadE3) -> Net-(P42-Pad1)
- J1 pad E30: Net-(J1-PadE30) -> Net-(P55-Pad1)
- J1 pad E6: (no net) -> unconnected-(J1-PadE6)
- J1 pad E8: Net-(J1-PadE8) -> Net-(P90-Pad1)
- P1 pad 1: Net-(J1-PadA10) -> (no net)
- P10 pad 1: Net-(J1-PadC2) -> (no net)
- P11 pad 1: Net-(J1-PadC3) -> (no net)
- P12 pad 1: Net-(J1-PadC4) -> (no net)
- P13 pad 1: Net-(J1-PadC5) -> (no net)
- P14 pad 1: Net-(J1-PadC6) -> (no net)
- P15 pad 1: Net-(J1-PadC7) -> (no net)
- P16 pad 1: Net-(J1-PadC8) -> (no net)
- P17 pad 1: Net-(J1-PadC9) -> (no net)
- P18 pad 1: Net-(J1-PadC10) -> (no net)
- P19 pad 1: Net-(J1-PadC11) -> (no net)
- P2 pad 1: Net-(J1-PadA28) -> (no net)
- P20 pad 1: Net-(J1-PadC12) -> (no net)
- P21 pad 1: Net-(J1-PadC13) -> (no net)
- P22 pad 1: Net-(J1-PadC14) -> (no net)
- P23 pad 1: Net-(J1-PadC15) -> (no net)
- P24 pad 1: Net-(J1-PadC16) -> (no net)
- P25 pad 1: Net-(J1-PadC17) -> (no net)
- P26 pad 1: Net-(J1-PadC18) -> (no net)
- P27 pad 1: Net-(J1-PadC19) -> (no net)
- P28 pad 1: Net-(J1-PadC20) -> (no net)
- P29 pad 1: Net-(J1-PadC21) -> (no net)
- P3 pad 1: Net-(J1-PadA31) -> (no net)
- P30 pad 1: Net-(J1-PadC22) -> (no net)
- P31 pad 1: Net-(J1-PadD2) -> (no net)
- P32 pad 1: Net-(J1-PadD3) -> (no net)
- P33 pad 1: Net-(J1-PadD5) -> (no net)
- P34 pad 1: Net-(J1-PadD6) -> (no net)
- P35 pad 1: Net-(J1-PadD8) -> (no net)
- P36 pad 1: Net-(J1-PadD9) -> (no net)
- P37 pad 1: Net-(J1-PadD10) -> (no net)
- P38 pad 1: Net-(J1-PadD12) -> (no net)
- P39 pad 1: Net-(J1-PadD15) -> (no net)
- P4 pad 1: Net-(J1-PadB10) -> (no net)
- P40 pad 1: Net-(J1-PadE1) -> (no net)
- P41 pad 1: Net-(J1-PadE2) -> (no net)
- P42 pad 1: Net-(J1-PadE3) -> (no net)
- P43 pad 1: Net-(J1-PadE12) -> (no net)
- P44 pad 1: Net-(J1-PadE13) -> (no net)
- P45 pad 1: Net-(J1-PadE15) -> (no net)
- P46 pad 1: Net-(J1-PadE16) -> (no net)
- P47 pad 1: Net-(J1-PadE18) -> (no net)
- P48 pad 1: Net-(J1-PadE20) -> (no net)
- P49 pad 1: Net-(J1-PadE21) -> (no net)
- P5 pad 1: Net-(J1-PadB13) -> (no net)
- P50 pad 1: Net-(J1-PadE23) -> (no net)
- P51 pad 1: Net-(J1-PadE25) -> (no net)
- P52 pad 1: Net-(J1-PadE26) -> (no net)
- P53 pad 1: Net-(J1-PadE27) -> (no net)
- P54 pad 1: Net-(J1-PadE29) -> (no net)
- P55 pad 1: Net-(J1-PadE30) -> (no net)
- P6 pad 1: Net-(J1-PadB18) -> (no net)
- P7 pad 1: Net-(J1-PadB19) -> (no net)
- P8 pad 1: Net-(J1-PadB20) -> (no net)
- P89 pad 1: Net-(J1-PadB21) -> (no net)
- P9 pad 1: Net-(J1-PadC1) -> (no net)
- P90 pad 1: Net-(J1-PadE8) -> (no net)
- P91 pad 1: Net-(J1-PadE14) -> (no net)
- P92 pad 1: Net-(J1-PadE19) -> (no net)
Routing:
- net /5V_SENSOR_1: track 245.3 -> 0.00 mm, vias 2 -> 0
- net /DIGITAL_3: track 181.2 -> 0.00 mm, vias 1 -> 0
- net /DIGITAL_2: track 179.3 -> 0.00 mm, vias 1 -> 0
- net /AV7: track 177.3 -> 0.00 mm, vias 1 -> 0
- net /DIGITAL_4: track 173.3 -> 0.00 mm, vias 1 -> 0
- net /DIGITAL_1: track 170.1 -> 0.00 mm, vias 1 -> 0
- net /AV3: track 167.7 -> 0.00 mm, vias 1 -> 0
- net /IN_KNOCK: track 163.6 -> 0.00 mm, vias 2 -> 0
- net /LS5: track 155.5 -> 0.00 mm, vias 3 -> 0
- net /LS9: track 154.8 -> 0.00 mm, vias 3 -> 0
- net /LS6: track 152.0 -> 0.00 mm, vias 2 -> 0
- net /CAN+: track 148.3 -> 0.00 mm
- net /AV1: track 147.3 -> 0.00 mm, vias 1 -> 0
- net /AV2: track 146.7 -> 0.00 mm, vias 1 -> 0
- net /CAN-: track 139.3 -> 0.00 mm, vias 2 -> 0
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Other:
- board text added: "https://rusefi.com/s/proteus-honda125"

Commit message: Proteus-compatible board preview
Parts:
- removed P64, P97: Pad, hellen-one-common:PAD-TH
- added F3: Fuse-Pad-Pad, hellen-one-common:PAD-1206-PAD, F.Cu at (135.5, 100.1)
- added G6: RUSEFI_LOGO, kicad6-libraries:rusefi_logo, F.Cu at (206.5, 210.3)
- added G7: PROTO_AREA, hellen-one-common:PROTO_AREA, F.Cu at (115.3, 202.6)
- added G8: PROTO_AREA, hellen-one-common:PROTO_AREA, F.Cu at (107.7, 215.3)
- M1: value Module-wbo-0.2 -> Module-wbo-0.3; footprint hellen-one-wbo-0.2:wbo -> hellen-one-wbo-0.3:wbo
- moved G1 187.2 mm to (122.9, 215.3), turned to 90 degrees
- moved G2 186.7 mm to (107.7, 202.6), turned to 90 degrees
- moved G3 185.0 mm to (130.6, 215.3), turned to 90 degrees
- moved P96 181.5 mm to (139.0, 166.8)
- moved G4 178.2 mm to (115.3, 215.3), turned to 90 degrees
- moved P94 178.0 mm to (139.0, 155.3), turned to 0 degrees
- moved P93 177.9 mm to (139.5, 145.8), turned to -90 degrees
- moved P95 177.3 mm to (139.5, 150.8), turned to -90 degrees
- moved P76 171.6 mm to (161.0, 190.8)
- moved P77 167.8 mm to (164.0, 190.8)
- moved P73 165.9 mm to (158.0, 190.8)
- moved P74 164.4 mm to (167.0, 190.8), turned to 0 degrees
- moved P75 161.0 mm to (170.0, 190.8), turned to 0 degrees
- moved G5 155.8 mm to (135.6, 197.5), turned to 180 degrees
- moved P59 127.9 mm to (203.3, 165.3), turned to 0 degrees
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- renumbered D2 to BRD1
Connections:
- BRD1 pad A1: (no net) -> Net-(P57-Pad1)
- BRD1 pad A10: (no net) -> /OUT_IAC
- BRD1 pad A11: (no net) -> /OUT_IMRC
- BRD1 pad A12: (no net) -> /OUT_VTS
- BRD1 pad A13: (no net) -> Net-(P58-Pad1)
- BRD1 pad A14: (no net) -> Net-(P59-Pad1)
- BRD1 pad A15: (no net) -> Net-(P61-Pad1)
- BRD1 pad A16: (no net) -> Net-(P63-Pad1)
- BRD1 pad A17: (no net) -> GND
- BRD1 pad A18: (no net) -> GND
- BRD1 pad A19: (no net) -> /OUT_INJ1
- BRD1 pad A2: (no net) -> Net-(P56-Pad1)
- BRD1 pad A20: (no net) -> /OUT_CHECK_ENGINE
- BRD1 pad A21: (no net) -> /OUT_MCS
- BRD1 pad A22: (no net) -> /OUT_IGN3
- BRD1 pad A23: (no net) -> /OUT_VTC
- BRD1 pad A24: (no net) -> GND
- BRD1 pad A25: (no net) -> Net-(P72-Pad1)
- BRD1 pad A26: (no net) -> Net-(P71-Pad1)
- BRD1 pad A27: (no net) -> Net-(P70-Pad1)
- BRD1 pad A28: (no net) -> Net-(P69-Pad1)
- BRD1 pad A29: (no net) -> Net-(P68-Pad1)
- BRD1 pad A3: (no net) -> Net-(P60-Pad1)
- BRD1 pad A30: (no net) -> Net-(P67-Pad1)
- BRD1 pad A31: (no net) -> Net-(P66-Pad1)
- BRD1 pad A32: (no net) -> Net-(P65-Pad1)
- BRD1 pad A33: (no net) -> /OUT_IGN4
- BRD1 pad A34: (no net) -> /OUT_IGN2
- BRD1 pad A35: (no net) -> /OUT_IGN1
- BRD1 pad A4: (no net) -> Net-(P62-Pad1)
- BRD1 pad A5: (no net) -> /OUT_INJ4
- BRD1 pad A6: (no net) -> /OUT_INJ3
- BRD1 pad A7: (no net) -> /OUT_INJ2
- BRD1 pad A8: (no net) -> /OUT_MAIN
- BRD1 pad A9: (no net) -> /OUT_FUEL_PUMP
- BRD1 pad B1: (no net) -> /IN_CRANK
- BRD1 pad B10: (no net) -> /IN_CAM2
- BRD1 pad B11: (no net) -> Net-(P73-Pad1)
- BRD1 pad B12: (no net) -> Net-(P77-Pad1)
- BRD1 pad B13: (no net) -> Net-(P75-Pad1)
- BRD1 pad B14: (no net) -> Net-(P82-Pad1)
- BRD1 pad B15: (no net) -> Net-(P80-Pad1)
- BRD1 pad B16: (no net) -> /CAN_L
- BRD1 pad B17: (no net) -> /CAN_H
- BRD1 pad B18: (no net) -> /IN_VIGN
- BRD1 pad B19: (no net) -> GND
- BRD1 pad B2: (no net) -> /IN_VSS
- BRD1 pad B20: (no net) -> GND
- BRD1 pad B21: (no net) -> Net-(P84-Pad1)
- BRD1 pad B22: (no net) -> Net-(P83-Pad1)
- BRD1 pad B23: (no net) -> /12V_MR
- BRD1 pad B3: (no net) -> /IN_CAM1
- BRD1 pad B4: (no net) -> Net-(P76-Pad1)
- BRD1 pad B5: (no net) -> Net-(P74-Pad1)
- BRD1 pad B6: (no net) -> Net-(P79-Pad1)
- BRD1 pad B7: (no net) -> Net-(P78-Pad1)
- BRD1 pad B8: (no net) -> Net-(P81-Pad1)
- BRD1 pad B9: (no net) -> /IN_VTPSW
- BRD1 pad C1: (no net) -> GND
- BRD1 pad C10: (no net) -> /5V_SENSOR_2
- BRD1 pad C11: (no net) -> /12V_PROT
- BRD1 pad C12: (no net) -> /12V_PROT
- BRD1 pad C13: (no net) -> /IN_PPS2
- BRD1 pad C14: (no net) -> /IN_TPS
- BRD1 pad C15: (no net) -> /IN_BRAKE
- BRD1 pad C16: (no net) -> Net-(P85-Pad1)
- BRD1 pad C17: (no net) -> Net-(P87-Pad1)
- BRD1 pad C18: (no net) -> Net-(P93-Pad1)
- BRD1 pad C19: (no net) -> /IN_IAT
- BRD1 pad C2: (no net) -> GND
- BRD1 pad C20: (no net) -> Net-(P94-Pad1)
- BRD1 pad C21: (no net) -> /5V_SENSOR_1
- BRD1 pad C22: (no net) -> /5V_SENSOR_2
- BRD1 pad C23: (no net) -> GND
- BRD1 pad C24: (no net) -> /IN_PPS1
- BRD1 pad C25: (no net) -> /IN_MRC
- BRD1 pad C26: (no net) -> /IN_MAP
- BRD1 pad C27: (no net) -> Net-(P86-Pad1)
- BRD1 pad C28: (no net) -> Net-(P88-Pad1)
- BRD1 pad C29: (no net) -> GND
- BRD1 pad C3: (no net) -> GND
- BRD1 pad C30: (no net) -> /IN_CLT
- BRD1 pad C31: (no net) -> Net-(P95-Pad1)
- BRD1 pad C32: (no net) -> /5V_SENSOR_1
- BRD1 pad C33: (no net) -> /5V_SENSOR_2
- BRD1 pad C34: (no net) -> /IN_KNOCK
- BRD1 pad C35: (no net) -> Net-(P96-Pad1)
- BRD1 pad C4: (no net) -> GND
- BRD1 pad C5: (no net) -> GND
- BRD1 pad C6: (no net) -> GND
- BRD1 pad C7: (no net) -> GND
- BRD1 pad C8: (no net) -> GND
- BRD1 pad C9: (no net) -> /5V_SENSOR_1
- J1 pad A10: Net-(P1-Pad1) -> Net-(J1-PadA10)
- J1 pad A11: /LS14 -> /OUT_IMRC
- J1 pad A12: /LS13 -> /OUT_IAC
- J1 pad A13: /IGN4 -> /OUT_IGN4
- J1 pad A14: /IGN3 -> /OUT_IGN3
- J1 pad A15: /IGN2 -> /OUT_IGN2
- J1 pad A16: /IGN1 -> /OUT_IGN1
- J1 pad A17: unconnected-(J1-PadA17) -> (no net)
- J1 pad A18: /DIGITAL_3 -> /IN_VSS
- J1 pad A19: /DIGITAL_4 -> /IN_CAM1
- J1 pad A22: unconnected-(J1-PadA22) -> (no net)
- J1 pad A25: /AV1 -> /IN_PPS2
- J1 pad A26: /AV2 -> /IN_PPS1
- J1 pad A27: unconnected-(J1-PadA27) -> (no net)
- J1 pad A28: Net-(P2-Pad1) -> Net-(J1-PadA28)
- J1 pad A29: /AV3 -> /IN_TPS
- J1 pad A30: /AV7 -> /IN_MAP
- J1 pad A31: Net-(P3-Pad1) -> Net-(J1-PadA31)
- J1 pad A6: /DIGITAL_1 -> /IN_CAM2
- J1 pad A7: /DIGITAL_2 -> /IN_CRANK
- J1 pad B1: /LS15 -> /OUT_VTC
- J1 pad B10: Net-(P4-Pad1) -> Net-(J1-PadB10)
- J1 pad B11: /DIGITAL_5 -> /IN_VTPSW
- J1 pad B12: unconnected-(J1-PadB12) -> (no net)
- J1 pad B13: Net-(P5-Pad1) -> Net-(J1-PadB13)
- J1 pad B14: unconnected-(J1-PadB14) -> (no net)
- J1 pad B16: unconnected-(J1-PadB16) -> (no net)
- J1 pad B17: /AT1 -> /IN_IAT
- J1 pad B18: Net-(P6-Pad1) -> Net-(J1-PadB18)
- J1 pad B19: Net-(P7-Pad1) -> Net-(J1-PadB19)
- J1 pad B2: /LS1 -> /OUT_INJ4
- J1 pad B20: Net-(P8-Pad1) -> Net-(J1-PadB20)
- J1 pad B21: Net-(P89-Pad1) -> Net-(J1-PadB21)
- J1 pad B22: /AV4 -> /IN_MRC
- J1 pad B23: unconnected-(J1-PadB23) -> (no net)
- J1 pad B24: unconnected-(J1-PadB24) -> (no net)
- J1 pad B3: /LS2 -> /OUT_INJ3
- J1 pad B4: /LS3 -> /OUT_INJ2
- J1 pad B5: /LS4 -> /OUT_INJ1
- J1 pad B6: /LS16 -> /OUT_VTS
- J1 pad B7: unconnected-(J1-PadB7) -> (no net)
- J1 pad B8: /AT2 -> /IN_CLT
- J1 pad B9: unconnected-(J1-PadB9) -> (no net)
- J1 pad C1: Net-(P9-Pad1) -> Net-(J1-PadC1)
- J1 pad C10: Net-(P18-Pad1) -> Net-(J1-PadC10)
- J1 pad C11: Net-(P19-Pad1) -> Net-(J1-PadC11)
- J1 pad C12: Net-(P20-Pad1) -> Net-(J1-PadC12)
- J1 pad C13: Net-(P21-Pad1) -> Net-(J1-PadC13)
- J1 pad C14: Net-(P22-Pad1) -> Net-(J1-PadC14)
- J1 pad C15: Net-(P23-Pad1) -> Net-(J1-PadC15)
- J1 pad C16: Net-(P24-Pad1) -> Net-(J1-PadC16)
- J1 pad C17: Net-(P25-Pad1) -> Net-(J1-PadC17)
- J1 pad C18: Net-(P26-Pad1) -> Net-(J1-PadC18)
- J1 pad C19: Net-(P27-Pad1) -> Net-(J1-PadC19)
- J1 pad C2: Net-(P10-Pad1) -> Net-(J1-PadC2)
- J1 pad C20: Net-(P28-Pad1) -> Net-(J1-PadC20)
- J1 pad C21: Net-(P29-Pad1) -> Net-(J1-PadC21)
- J1 pad C22: Net-(P30-Pad1) -> Net-(J1-PadC22)
- J1 pad C3: Net-(P11-Pad1) -> Net-(J1-PadC3)
- J1 pad C4: Net-(P12-Pad1) -> Net-(J1-PadC4)
- J1 pad C5: Net-(P13-Pad1) -> Net-(J1-PadC5)
- J1 pad C6: Net-(P14-Pad1) -> Net-(J1-PadC6)
- J1 pad C7: Net-(P15-Pad1) -> Net-(J1-PadC7)
- J1 pad C8: Net-(P16-Pad1) -> Net-(J1-PadC8)
- J1 pad C9: Net-(P17-Pad1) -> Net-(J1-PadC9)
- J1 pad D1: unconnected-(J1-PadD1) -> (no net)
- J1 pad D10: Net-(P37-Pad1) -> Net-(J1-PadD10)
- J1 pad D11: unconnected-(J1-PadD11) -> (no net)
- J1 pad D12: Net-(P38-Pad1) -> Net-(J1-PadD12)
- J1 pad D13: unconnected-(J1-PadD13) -> (no net)
- J1 pad D14: unconnected-(J1-PadD14) -> (no net)
- J1 pad D15: Net-(P39-Pad1) -> Net-(J1-PadD15)
- J1 pad D16: unconnected-(J1-PadD16) -> (no net)
- J1 pad D17: unconnected-(J1-PadD17) -> (no net)
- J1 pad D2: Net-(P31-Pad1) -> Net-(J1-PadD2)
- J1 pad D3: Net-(P32-Pad1) -> Net-(J1-PadD3)
- J1 pad D4: unconnected-(J1-PadD4) -> (no net)
- J1 pad D5: Net-(P33-Pad1) -> Net-(J1-PadD5)
- J1 pad D6: Net-(P34-Pad1) -> Net-(J1-PadD6)
- J1 pad D7: unconnected-(J1-PadD7) -> (no net)
- J1 pad D8: Net-(P35-Pad1) -> Net-(J1-PadD8)
- J1 pad D9: Net-(P36-Pad1) -> Net-(J1-PadD9)
- J1 pad E1: Net-(P40-Pad1) -> Net-(J1-PadE1)
- J1 pad E10: unconnected-(J1-PadE10) -> (no net)
- J1 pad E11: /CAN+ -> /CAN_H
- J1 pad E12: Net-(P43-Pad1) -> Net-(J1-PadE12)
- J1 pad E13: Net-(P44-Pad1) -> Net-(J1-PadE13)
- J1 pad E14: Net-(P91-Pad1) -> Net-(J1-PadE14)
- J1 pad E15: Net-(P45-Pad1) -> Net-(J1-PadE15)
- J1 pad E16: Net-(P46-Pad1) -> Net-(J1-PadE16)
- J1 pad E17: /LS9 -> /OUT_FUEL_PUMP
- J1 pad E18: Net-(P47-Pad1) -> Net-(J1-PadE18)
- J1 pad E19: Net-(P92-Pad1) -> Net-(J1-PadE19)
- J1 pad E2: Net-(P41-Pad1) -> Net-(J1-PadE2)
- J1 pad E20: Net-(P48-Pad1) -> Net-(J1-PadE20)
- J1 pad E21: Net-(P49-Pad1) -> Net-(J1-PadE21)
- J1 pad E22: /AV5 -> /IN_BRAKE
- J1 pad E23: Net-(P50-Pad1) -> Net-(J1-PadE23)
- J1 pad E24: /CAN- -> /CAN_L
- J1 pad E25: Net-(P51-Pad1) -> Net-(J1-PadE25)
- J1 pad E26: Net-(P52-Pad1) -> Net-(J1-PadE26)
- J1 pad E27: Net-(P53-Pad1) -> Net-(J1-PadE27)
- J1 pad E28: unconnected-(J1-PadE28) -> (no net)
- J1 pad E29: Net-(P54-Pad1) -> Net-(J1-PadE29)
- J1 pad E3: Net-(P42-Pad1) -> Net-(J1-PadE3)
- J1 pad E30: Net-(P55-Pad1) -> Net-(J1-PadE30)
- J1 pad E31: /LS6 -> /OUT_CHECK_ENGINE
- J1 pad E6: unconnected-(J1-PadE6) -> (no net)
- J1 pad E7: /LS5 -> /OUT_MAIN
- J1 pad E8: Net-(P90-Pad1) -> Net-(J1-PadE8)
- J1 pad E9: /12V_RAW -> Net-(J1-PadE9)
- M2 pad S1: /CAN- -> /CAN_L
- M2 pad S2: /CAN+ -> /CAN_H
- P1 pad 1: (no net) -> Net-(J1-PadA10)
- P10 pad 1: (no net) -> Net-(J1-PadC2)
- P11 pad 1: (no net) -> Net-(J1-PadC3)
- P12 pad 1: (no net) -> Net-(J1-PadC4)
- P13 pad 1: (no net) -> Net-(J1-PadC5)
- P14 pad 1: (no net) -> Net-(J1-PadC6)
- P15 pad 1: (no net) -> Net-(J1-PadC7)
- P16 pad 1: (no net) -> Net-(J1-PadC8)
- P17 pad 1: (no net) -> Net-(J1-PadC9)
- P18 pad 1: (no net) -> Net-(J1-PadC10)
- P19 pad 1: (no net) -> Net-(J1-PadC11)
- P2 pad 1: (no net) -> Net-(J1-PadA28)
- P20 pad 1: (no net) -> Net-(J1-PadC12)
- P21 pad 1: (no net) -> Net-(J1-PadC13)
- P22 pad 1: (no net) -> Net-(J1-PadC14)
- P23 pad 1: (no net) -> Net-(J1-PadC15)
- P24 pad 1: (no net) -> Net-(J1-PadC16)
- P25 pad 1: (no net) -> Net-(J1-PadC17)
- P26 pad 1: (no net) -> Net-(J1-PadC18)
- P27 pad 1: (no net) -> Net-(J1-PadC19)
- P28 pad 1: (no net) -> Net-(J1-PadC20)
- P29 pad 1: (no net) -> Net-(J1-PadC21)
- P3 pad 1: (no net) -> Net-(J1-PadA31)
- P30 pad 1: (no net) -> Net-(J1-PadC22)
- P31 pad 1: (no net) -> Net-(J1-PadD2)
- P32 pad 1: (no net) -> Net-(J1-PadD3)
- P33 pad 1: (no net) -> Net-(J1-PadD5)
- P34 pad 1: (no net) -> Net-(J1-PadD6)
- P35 pad 1: (no net) -> Net-(J1-PadD8)
- P36 pad 1: (no net) -> Net-(J1-PadD9)
- P37 pad 1: (no net) -> Net-(J1-PadD10)
- P38 pad 1: (no net) -> Net-(J1-PadD12)
- P39 pad 1: (no net) -> Net-(J1-PadD15)
- P4 pad 1: (no net) -> Net-(J1-PadB10)
- P40 pad 1: (no net) -> Net-(J1-PadE1)
- P41 pad 1: (no net) -> Net-(J1-PadE2)
- P42 pad 1: (no net) -> Net-(J1-PadE3)
- P43 pad 1: (no net) -> Net-(J1-PadE12)
- P44 pad 1: (no net) -> Net-(J1-PadE13)
- P45 pad 1: (no net) -> Net-(J1-PadE15)
- P46 pad 1: (no net) -> Net-(J1-PadE16)
- P47 pad 1: (no net) -> Net-(J1-PadE18)
- P48 pad 1: (no net) -> Net-(J1-PadE20)
- P49 pad 1: (no net) -> Net-(J1-PadE21)
- P5 pad 1: (no net) -> Net-(J1-PadB13)
- P50 pad 1: (no net) -> Net-(J1-PadE23)
- P51 pad 1: (no net) -> Net-(J1-PadE25)
- P52 pad 1: (no net) -> Net-(J1-PadE26)
- P53 pad 1: (no net) -> Net-(J1-PadE27)
- P54 pad 1: (no net) -> Net-(J1-PadE29)
- P55 pad 1: (no net) -> Net-(J1-PadE30)
- P56 pad 1: /AT4 -> Net-(P56-Pad1)
- P57 pad 1: /5V_SENSOR_1 -> Net-(P57-Pad1)
- P58 pad 1: /5V_SENSOR_2 -> Net-(P58-Pad1)
- P59 pad 1: /KNOCK_2 -> Net-(P59-Pad1)
- P6 pad 1: (no net) -> Net-(J1-PadB18)
- P60 pad 1: /AT3 -> Net-(P60-Pad1)
- P61 pad 1: /HS2 -> Net-(P61-Pad1)
- P62 pad 1: /HS1 -> Net-(P62-Pad1)
- P63 pad 1: /LS11 -> Net-(P63-Pad1)
- P65 pad 1: /HS4 -> Net-(P65-Pad1)
- P66 pad 1: /IGN12 -> Net-(P66-Pad1)
- P67 pad 1: /IGN11 -> Net-(P67-Pad1)
- P68 pad 1: /IGN10 -> Net-(P68-Pad1)
- P69 pad 1: /IGN9 -> Net-(P69-Pad1)
- P7 pad 1: (no net) -> Net-(J1-PadB19)
- P70 pad 1: /IGN8 -> Net-(P70-Pad1)
- P71 pad 1: /IGN7 -> Net-(P71-Pad1)
- P72 pad 1: /IGN6 -> Net-(P72-Pad1)
- P73 pad 1: /IGN5 -> Net-(P73-Pad1)
- P74 pad 1: /AV9 -> Net-(P74-Pad1)
- P75 pad 1: /AV11 -> Net-(P75-Pad1)
- P76 pad 1: /AV8 -> Net-(P76-Pad1)
- P77 pad 1: /AV10 -> Net-(P77-Pad1)
- P78 pad 1: /VR2+ -> Net-(P78-Pad1)
- P79 pad 1: /VR1+ -> Net-(P79-Pad1)
- P8 pad 1: (no net) -> Net-(J1-PadB20)
- P80 pad 1: /ETB1- -> Net-(P80-Pad1)
- P81 pad 1: /ETB1+ -> Net-(P81-Pad1)
- P82 pad 1: /ETB2- -> Net-(P82-Pad1)
- P83 pad 1: /DIGITAL_6 -> Net-(P83-Pad1)
- P84 pad 1: /VR2- -> Net-(P84-Pad1)
- P85 pad 1: /VR1- -> Net-(P85-Pad1)
- P86 pad 1: /ETB2+ -> Net-(P86-Pad1)
- P87 pad 1: /CAN2- -> Net-(P87-Pad1)
- P88 pad 1: /CAN2+ -> Net-(P88-Pad1)
- P89 pad 1: (no net) -> Net-(J1-PadB21)
- P9 pad 1: (no net) -> Net-(J1-PadC1)
- P90 pad 1: (no net) -> Net-(J1-PadE8)
- P91 pad 1: (no net) -> Net-(J1-PadE14)
- P92 pad 1: (no net) -> Net-(J1-PadE19)
- P93 pad 1: /LS7 -> Net-(P93-Pad1)
- P94 pad 1: /LS8 -> Net-(P94-Pad1)
- P95 pad 1: /LS10 -> Net-(P95-Pad1)
- P96 pad 1: /LS12 -> Net-(P96-Pad1)
Routing:
- net /5V_SENSOR_1: track 0.00 -> 269.0 mm, vias 0 -> 2
- net /CAN_H: track 0.00 -> 177.2 mm, vias 0 -> 2
- net /CAN_L: track 0.00 -> 167.0 mm
- net /IN_MAP: track 0.00 -> 161.7 mm, vias 0 -> 2
- net /IN_TPS: track 0.00 -> 160.4 mm, vias 0 -> 2
- net /IN_KNOCK: track 0.00 -> 158.1 mm, vias 0 -> 2
- net /IN_CRANK: track 0.00 -> 156.4 mm, vias 0 -> 2
- net /IN_VSS: track 0.00 -> 156.1 mm, vias 0 -> 2
- net /IN_CAM1: track 0.00 -> 154.6 mm, vias 0 -> 2
- net /OUT_FUEL_PUMP: track 0.00 -> 153.7 mm, vias 0 -> 1
- net /OUT_MAIN: track 0.00 -> 152.3 mm, vias 0 -> 1
- net /IN_CAM2: track 0.00 -> 146.2 mm, vias 0 -> 2
- net /IN_PPS2: track 0.00 -> 141.8 mm, vias 0 -> 2
- net /OUT_CHECK_ENGINE: track 0.00 -> 138.9 mm, vias 0 -> 2
- net /IN_PPS1: track 0.00 -> 138.5 mm, vias 0 -> 2
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Other:
- board text added: "12V"
- board text added: "5V"
- board text added: "GND"
