File: proteus125honda.kicad_pcb (KiCad board)
At the start: 2 copper layers, 153 x 151.3 mm, 121 parts, among them J1 1318612-1, J10 Conn_01x01, J11 Conn_01x01, J12 Conn_01x01, J13 Conn_01x01, J2 XH-8A, J3 Conn_01x06, J7 Conn_01x01, J8 Conn_01x01, J9 Conn_01x01, M1 Module-wbo-0.3, M2 Module-can-0.1, P1 Pad, P10 Pad, P11 Pad, P12 Pad, P13 Pad, P14 Pad, P15 Pad, P16 Pad, P17 Pad, P18 Pad, P19 Pad, P2 Pad, P20 Pad, P21 Pad, P22 Pad, P23 Pad, P24 Pad, P25 Pad, P26 Pad, P27 Pad, P28 Pad, P29 Pad, P3 Pad, P30 Pad, P31 Pad, P32 Pad, P33 Pad, P34 Pad, P35 Pad, P36 Pad, P37 Pad, P38 Pad, P39 Pad, P4 Pad, P40 Pad, P41 Pad, P42 Pad, P43 Pad, P44 Pad, P45 Pad, P46 Pad, P47 Pad, P48 Pad, P49 Pad, P5 Pad, P50 Pad, P51 Pad, P52 Pad, P53 Pad, P54 Pad, P55 Pad, P56 Pad, P57 Pad, P58 Pad, P59 Pad, P6 Pad, P60 Pad, P61 Pad, P62 Pad, P63 Pad, P65 Pad, P66 Pad, P67 Pad, P68 Pad, P69 Pad, P7 Pad, P70 Pad, P71 Pad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

Commit message: #10
Other:
- board text added: "1 2 IGN 3 4"
- board text added: "1 2 INJ 3 4"
- board text added: "12V_MR"
- board text added: "BRAKE"
- board text added: "CAM1"
- board text added: "CAM2"
- board text added: "CAN H"
- board text added: "CAN L"
- board text added: "CLT"
- board text added: "CRANK"
- board text added: "IAC"
- board text added: "IAT"
- board text added: "IMRC"
- board text added: "KNOCK"
- board text added: "MAIN"
- board text added: "MAP"
- board text added: "MCS"
- board text added: "MRC"
- board text added: "PPS2"
- board text added: "PSP1"
- board text added: "TPS"
- board text added: "VIGN"
- board text added: "VTC"
- board text added: "VTPSW"
- board text added: "VTS"
Changed lines of the file:
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@@
   (gr_line (start 248 206.8) (end 248 150.8) (layer "Edge.Cuts") (width 0.2))
   (gr_arc (start 244.000001 77.5) (end 248 77.5) (angle -90) (layer "Edge.Cuts") (width 0.2))
+  (gr_text "KNOCK" (at 208.3 88.4 90) (layer "B.SilkS")
+    (effects (font (size 1 1) (thickness 0.15)) (justify mirror))
+  )
+  (gr_text "CAN L" (at 113.1 72.9 90) (layer "B.SilkS")
+    (effects (font (size 1 1) (thickness 0.15)) (justify mirror))
+  )
+  (gr_text "IAC" (at 214.8 80.6) (layer "B.SilkS")
+    (effects (font (size 1 1) (thickness 0.15)) (justify mirror))
+  )
+  (gr_text "5V" (at 236.3 80.7) (layer "B.SilkS")
+    (effects (font (size 1 1) (thickness 0.15)) (justify mirror))
+  )
+  (gr_text "1 2 IGN 3 4" (at 221.2 80.6) (layer "B.SilkS")
+    (effects (font (size 1 1) (thickness 0.15)) (justify mirror))
+  )
+  (gr_text "1 2 INJ 3   4" (at 192.6 90.2) (layer "B.SilkS")
+    (effects (font (size 1 1) (thickness 0.15)) (justify mirror))
+  )
+  (gr_text "PSP1" (at 221 73.4 90) (layer "B.SilkS")
+    (effects (font (size 1 1) (thickness 0.15)) (justify mirror))
+  )
   (gr_text "5V" (at 138.8 194.94) (layer "B.SilkS")
     (effects (font (size 1 1) (thickness 0.15)) (justify left mirror))
+  )
+  (gr_text "CAN H" (at 110.1 80.6) (layer "B.SilkS")
+    (effects (font (size 1 1) (thickness 0.15)) (justify mirror))
+  )
+  (gr_text "12V_MR" (at 216.1 90.2) (layer "B.SilkS")
+    (effects (font (size 1 1) (thickness 0.15)) (justify mirror))
+  )
+  (gr_text "IAT" (at 181.9 78.6) (layer "B.SilkS")
+    (effects (font (size 1 1) (thickness 0.15)) (justify mirror))
+  )
+  (gr_text "GND" (at 119.5 90.2) (layer "B.SilkS")
+    (effects (font (size 1 1) (thickness 0.15)) (justify mirror))
+  )
+  (gr_text "VTS" (at 201.5 91.1 90) (layer "B.SilkS")
+    (effects (font (size 1 1) (thickness 0.15)) (justify mirror))
+  )
+  (gr_text "PPS2" (at 218.4 73.4 90) (layer "B.SilkS")
+    (effects (font (size 1 1) (thickness 0.15)) (justify mirror))
+  )
+  (gr_text "VTC" (at 183.8 91.3 90) (layer "B.SilkS")
+    (effects (font (size 1 1) (thickness 0.15)) (justify mirror))
+  )
+  (gr_text "TPS" (at 235.2 73.5 90) (layer "B.SilkS")
+    (effects (font (size 1 1) (thickness 0.15)) (justify mirror))
+  )
+  (gr_text "MAP" (at 237.4 73.5 90) (layer "B.SilkS")
+    (effects (font (size 1 1) (thickness 0.15)) (justify mirror))
+  )
+  (gr_text "CAM2" (at 228.3 91.7 90) (layer "B.SilkS")
+    (effects (font (size 1 1) (thickness 0.15)) (justify mirror))
+  )
+  (gr_text "VTPSW" (at 191.8 80.5) (layer "B.SilkS")
+    (effects (font (size 1 1) (thickness 0.15)) (justify mirror))
+  )
+  (gr_text "MAIN" (at 129 90.2) (layer "B.SilkS")
+    (effects (font (size 1 1) (thickness 0.15)) (justify mirror))
+  )
+  (gr_text "GND" (at 213.8 74.2) (layer "B.SilkS")
+    (effects (font (size 1 1) (thickness 0.15)) (justify mirror))
+  )
+  (gr_text "CRANK" (at 231.5 92 90) (layer "B.SilkS")
+    (effects (font (size 1 1) (thickness 0.15)) (justify mirror))
+  )
+  (gr_text "GND" (at 236.2 88.3 90) (layer "B.SilkS")
+    (effects (font (size 1 1) (thickness 0.15)) (justify mirror))
+  )
+  (gr_text "CAM1" (at 232.4 80.5) (layer "B.SilkS")
+    (effects (font (size 1 1) (thickness 0.15)) (justify mirror))
+  )
+  (gr_text "CLT" (at 181.6 82.2) (layer "B.SilkS")
+    (effects (font (size 1 1) (thickness 0.15)) (justify mirror))
+  )
+  (gr_text "MCS" (at 201.7 80.5) (layer "B.SilkS")
+    (effects (font (size 1 1) (thickness 0.15)) (justify mirror))
+  )
+  (gr_text "BRAKE" (at 107.9 73 90) (layer "B.SilkS")
+    (effects (font (size 1 1) (thickness 0.15)) (justify mirror))
+  )
+  (gr_text "IMRC" (at 211.9 80.6) (layer "B.SilkS")
+    (effects (font (size 1 1) (thickness 0.15)) (justify mirror))
+  )
+  (gr_text "MRC" (at 200.2 74.1 90) (layer "B.SilkS")
+    (effects (font (size 1 1) (thickness 0.15)) (justify mirror))
   )
   (gr_text "GND" (at 139.853618 197.5) (layer "B.SilkS")
     (effects (font (size 1 1) (thickness 0.15)) (justify left mirror))
   )
+  (gr_text "VIGN" (at 137.7 85.2) (layer "B.SilkS")
+    (effects (font (size 1 1) (thickness 0.15)) (justify mirror))
+  )
+  (gr_text "GND" (at 223.7 88.2 90) (layer "B.SilkS")
+    (effects (font (size 1 1) (thickness 0.15)) (justify mirror))
+  )
   (gr_text "12V" (at 139.853618 192.3) (layer "B.SilkS")
