File: proteus125honda.kicad_pcb (KiCad board)
At the start: 2 copper layers, 153 x 151.3 mm, 121 parts, among them J1 1318612-1, J10 Conn_01x01, J11 Conn_01x01, J12 Conn_01x01, J13 Conn_01x01, J2 XH-8A, J3 Conn_01x06, J7 Conn_01x01, J8 Conn_01x01, J9 Conn_01x01, M1 Module-wbo-0.3, M2 Module-can-0.1, P1 Pad, P10 Pad, P11 Pad, P12 Pad, P13 Pad, P14 Pad, P15 Pad, P16 Pad, P17 Pad, P18 Pad, P19 Pad, P2 Pad, P20 Pad, P21 Pad, P22 Pad, P23 Pad, P24 Pad, P25 Pad, P26 Pad, P27 Pad, P28 Pad, P29 Pad, P3 Pad, P30 Pad, P31 Pad, P32 Pad, P33 Pad, P34 Pad, P35 Pad, P36 Pad, P37 Pad, P38 Pad, P39 Pad, P4 Pad, P40 Pad, P41 Pad, P42 Pad, P43 Pad, P44 Pad, P45 Pad, P46 Pad, P47 Pad, P48 Pad, P49 Pad, P5 Pad, P50 Pad, P51 Pad, P52 Pad, P53 Pad, P54 Pad, P55 Pad, P56 Pad, P57 Pad, P58 Pad, P59 Pad, P6 Pad, P60 Pad, P61 Pad, P62 Pad, P63 Pad, P65 Pad, P66 Pad, P67 Pad, P68 Pad, P69 Pad, P7 Pad, P70 Pad, P71 Pad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

Commit message: MAP
Parts:
- removed P85: Pad, hellen-one-common:PAD-TH
- added C1: 100n, hellen-one-common:C0603, F.Cu at (146.5, 189.8)
- added C2: 47p, hellen-one-common:C0603, F.Cu at (143.4, 189.8)
- added R1: 51k, hellen-one-common:R0603, F.Cu at (143.4, 188.1)
- added U1: MPXxx6115A, kicad6-libraries:MPX_SOP_SSOP, F.Cu at (146.1, 201.4)
- moved G6 41.3 mm to (243.6, 192.2)
- moved M2 11.4 mm to (154.3, 192.9)
- moved M1 11.4 mm to (163.2, 207.9)
- moved J2 11.4 mm to (207.7, 202.5)
- moved G*** 2.50 mm to (226.5, 201.3)
- moved J3 1.29 mm to (164.7, 213.1)
Routing:
- net Net-(BRD1-PadC16): track 18.4 -> 82.2 mm, vias 0 -> 1
- net /5V_SENSOR_2: track 89.0 -> 113.2 mm, vias 0 -> 1
- net Net-(J3-Pad1): track 16.3 -> 9.08 mm
- net Net-(J3-Pad2): track 16.5 -> 10.0 mm
- net Net-(J3-Pad5): track 11.1 -> 16.9 mm
- net /CAN_L: track 167.0 -> 161.4 mm
- net /CAN_H: track 177.2 -> 172.8 mm, vias 2 -> 1
- net unconnected-(U1-Pad1): track 0.00 -> 4.34 mm
- net unconnected-(U1-Pad5): track 0.00 -> 4.16 mm
- net unconnected-(U1-Pad8): track 0.00 -> 4.15 mm
- net unconnected-(U1-Pad6): track 0.00 -> 3.63 mm
- net unconnected-(U1-Pad7): track 0.00 -> 3.63 mm
- net Net-(J3-Pad4): track 12.5 -> 14.1 mm
- net GND: vias 6 -> 7
Other:
- board text added: "C"
- board text added: "D"
- board text added: "G"
- board text added: "H-"
- board text added: "Ip"
- board text added: "R_Trim"
- board text added: "SWD:R"
- board text added: "V"
- board text added: "Vs"
- board text added: "Vs/Ip"
- board text added: "WBO1"

Commit message: Fix proteus
Parts:
- removed P84: Pad, hellen-one-common:PAD-TH
- moved P83 9.00 mm to (173.0, 190.8)
- moved P82 3.00 mm to (182.0, 190.8)
Connections:
- BRD1 pad B14: Net-(BRD1-PadB14) -> GND
- P82 pad 1: Net-(BRD1-PadB14) -> Net-(BRD1-PadB22)
- P83 pad 1: Net-(BRD1-PadB22) -> Net-(BRD1-PadB21)
Routing:
- net Net-(BRD1-PadB14): track 21.2 -> 0.00 mm

Commit message: Export
Parts:
- removed P39, P4, P5, P59, P62, P63: Pad, hellen-one-common:PAD-TH
- added R2: Jumper-Pad-Pad, hellen-one-common:PAD-0805-PAD, F.Cu at (198.6, 94.8)
- added R3: Jumper-Pad-Pad, hellen-one-common:PAD-0805-PAD, F.Cu at (189.5, 94.1)
- J2: value XH-8A -> XH-10A; footprint hellen-one-common:XH-8A -> Connector_Molex:Molex_SPOX_5267-10A_1x10_P2.50mm_Vertical
- moved P57 54.2 mm to (203.3, 129.3), turned to 90 degrees
- moved P56 48.0 mm to (203.3, 132.3), turned to 90 degrees
- moved P1 28.3 mm to (238.0, 97.8)
- moved P40 27.0 mm to (135.0, 93.8)
- moved P49 27.0 mm to (108.0, 93.8)
- moved P3 26.5 mm to (210.0, 93.8)
- moved F3 25.6 mm to (110.0, 102.8), turned to 0 degrees
- moved P41 24.4 mm to (132.0, 93.8)
- moved P50 24.4 mm to (132.0, 98.3)
- moved P90 24.4 mm to (108.0, 98.3)
- moved F1 21.5 mm to (235.0, 96.3)
- moved P48 21.0 mm to (111.0, 98.3)
- moved P15 21.0 mm to (158.5, 93.8)
- moved P16 21.0 mm to (179.5, 98.3)
- moved P23 21.0 mm to (158.5, 98.3)
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Connections:
- BRD1 pad A1: Net-(BRD1-PadA1) -> /OUT_VTC
- BRD1 pad A10: /OUT_IAC -> Net-(BRD1-PadA10)
- BRD1 pad A11: /OUT_IMRC -> Net-(BRD1-PadA11)
- BRD1 pad A12: /OUT_VTS -> /OUT_IAC
- BRD1 pad A14: Net-(BRD1-PadA14) -> /OUT_ALTRN_CONTROL
- BRD1 pad A16: Net-(BRD1-PadA16) -> /OUT_ETB_RELAY
- BRD1 pad A2: Net-(BRD1-PadA2) -> /OUT_VTS
- BRD1 pad A23: /OUT_VTC -> /OUT_IMRC
- BRD1 pad A4: Net-(BRD1-PadA4) -> /OUT_CHARGING_LIGHT
- J1 pad D15: Net-(J1-PadD15) -> /OUT_ETB_RELAY
- P56 pad 1: Net-(BRD1-PadA2) -> Net-(BRD1-PadA10)
- P57 pad 1: Net-(BRD1-PadA1) -> Net-(BRD1-PadA11)
Routing:
- net /OUT_ETB_RELAY: track 0.00 -> 141.9 mm, vias 0 -> 3
- net /OUT_ALTRN_CONTROL: track 0.00 -> 99.9 mm, vias 0 -> 1
- net /12V_MR: track 93.4 -> 179.1 mm, vias 0 -> 3
- net /OUT_CHARGING_LIGHT: track 0.00 -> 79.8 mm, vias 0 -> 1
- net /OUT_VTS: track 61.3 -> 121.9 mm, vias 2 -> 1
- net /OUT_VTC: track 76.8 -> 115.6 mm, vias 2 -> 1
- net /OUT_CHECK_ENGINE: track 138.9 -> 171.0 mm
- net /5V_SENSOR_1: track 269.0 -> 238.1 mm
- net Net-(BRD1-PadA4): track 29.0 -> 0.00 mm
- net /CAN_L: track 161.4 -> 133.4 mm
- net /IN_VIGN: track 93.5 -> 121.0 mm
- net /IN_KNOCK: track 158.1 -> 184.2 mm
- net Net-(J1-PadD15): track 25.9 -> 0.00 mm
- net Net-(BRD1-PadA16): track 25.6 -> 0.00 mm
- net /CAN_H: track 172.8 -> 147.5 mm
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Other:
- board text added: "+12V"
- board text added: "4 3 IGN 2 1"
- board text added: "4 3 INJ 2 1"
- board text added: "Always looking for C/C++/PHP/Java developers https://rusefi.com/s/mission"
- board text added: "Proteus Honda K-125 adapter rev. a"
- board text added: "VSS"
- board text removed: "1 2 IGN 3 4"
- board text removed: "1 2 INJ 3 4"
