File: proteus125honda.kicad_pcb (KiCad board)
At the start: 2 copper layers, 153 x 151.3 mm, 119 parts, among them J1 1318612-1, J10 Conn_01x01, J11 Conn_01x01, J12 Conn_01x01, J13 Conn_01x01, J2 XH-10A, J3 Conn_01x06, J7 Conn_01x01, J8 Conn_01x01, J9 Conn_01x01, M1 Module-wbo-0.3, M2 Module-can-0.1, P1 Pad, P10 Pad, P11 Pad, P12 Pad, P13 Pad, P14 Pad, P15 Pad, P16 Pad, P17 Pad, P18 Pad, P19 Pad, P2 Pad, P20 Pad, P21 Pad, P22 Pad, P23 Pad, P24 Pad, P25 Pad, P26 Pad, P27 Pad, P28 Pad, P29 Pad, P3 Pad, P30 Pad, P31 Pad, P32 Pad, P33 Pad, P34 Pad, P35 Pad, P36 Pad, P37 Pad, P38 Pad, P40 Pad, P41 Pad, P42 Pad, P43 Pad, P44 Pad, P45 Pad, P46 Pad, P47 Pad, P48 Pad, P49 Pad, P50 Pad, P51 Pad, P52 Pad, P53 Pad, P54 Pad, P55 Pad, P56 Pad, P57 Pad, P58 Pad, P6 Pad, P60 Pad, P61 Pad, P65 Pad, P66 Pad, P67 Pad, P68 Pad, P69 Pad, P7 Pad, P70 Pad, P71 Pad, P72 Pad, P73 Pad, P74 Pad, P75 Pad, P76 Pad, P77 Pad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

Commit message: #17, #18, #14, #13
Parts:
- removed J2: XH-10A, Connector_Molex:Molex_SPOX_5267-10A_1x10_P2.50mm_Vertical
- added D2: D_Schottky, Diode_SMD:D_SMA, F.Cu at (206.5, 98.7)
- added D3: DNP, Diode_SMD:D_SMA, F.Cu at (189.0, 98.8)
- added J4: XH-10AW, Connector_JST:JST_XH_S10B-XH-A_1x10_P2.50mm_Horizontal, F.Cu at (212.6, 195.2)
- added R4: Jumper-Pad-Pad, hellen-one-common:PAD-0805-PAD, F.Cu at (233.2, 101.7)
- G***: moved to B.Cu
- moved G*** 93.6 mm to (155.7, 140.1), turned to 180 degrees
- moved D1 0.20 mm to (189.0, 102.5)
Connections:
- J1 pad A12: /OUT_IAC -> Net-(J1-PadA12)
Routing:
- net /12V_MR: track 179.1 -> 230.7 mm, vias 3 -> 4
- net /WBO_H-: track 9.28 -> 40.2 mm
- net /WBO_R_Trim: track 5.39 -> 32.9 mm
- net /WBO_Ip: track 4.76 -> 30.2 mm
- net /WBO_Vs/Ip: track 5.16 -> 27.6 mm
- net /OUT_IAC: track 49.5 -> 27.7 mm
- net /WBO_Vs: track 5.78 -> 24.9 mm
- net GND: vias 243 -> 241
