File: proteus125honda.kicad_sch (KiCad schematic)
At the start: 4 parts, among them J1 1318612-1, J2 Conn_01x35, J3 Conn_01x35, J4 Conn_01x23

Commit message: Upd pinout
Parts:
- added ALTC, ALTF, ALTL, ATPP, ATPR, D3, D? (x19), SEDF, SEFD: Pad, hellen-one-common:PAD-TH, symbol hellen-one-common:Pad
- added D2, D? (x17): S-MODE, hellen-one-common:PAD-TH, symbol hellen-one-common:Pad
- added D?: D_Schottky, Diode_SMD:D_SMA, symbol Device:D_Schottky
- added J?: Conn_01x06, Connector_PinHeader_2.54mm:PinHeader_1x06_P2.54mm_Vertical, symbol Connector_Generic:Conn_01x06
- added M?: Module-wbo-0.2, hellen-one-wbo-0.2:wbo, symbol hellen-one-wbo-0.2:Module-wbo-0.2
- added M?: Module-can-0.1, hellen-one-can-0.1:can, symbol hellen-one-can-0.1:Module-can-0.1
Connections:
- net KNOCK_1 is gone; now on net IN_KNOCK: J3.34 (Pin_34)
- net 12V_MR: now also J1.A2, J1.A3, D?.1 (K)
- net 5V_SENSOR_1: now also J1.A20, J1.A21, J1.E5
- net AT1: now also J1.B17
- net AT2: now also J1.B8
- net AV1: now also J1.A25
- net AV2: now also J1.A26
- net AV3: now also J1.A29
- net AV4: now also J1.B22
- net DIGITAL_1: now also J1.A6
- net DIGITAL_2: now also J1.A7
- net DIGITAL_3: now also J1.A18
- net DIGITAL_4: now also J1.A19
- net DIGITAL_5: now also J1.B11
- net GND: now also J1.A23, J1.A24, J1.A4, J1.A5, J1.A8, J1.A9, J1.E4, J?.3 (Pin_3)
- net IGN1: now also J1.A16
- net IGN2: now also J1.A15
- net IGN3: now also J1.A14
- net IGN4: now also J1.A13
- net LS1: now also J1.B2
- net LS13: now also J1.A12
- net LS14: now also J1.A11
- net LS15: now also J1.B1
- net LS16: now also J1.B6
- net LS3: now also J1.B4
- net IN_KNOCK: now reaches J1.A1
- net at J1.C1: now also D?.1 (Pin_1)
- net at J1.C10: now also D?.1 (Pin_1)
- net at J1.C11: now also D?.1 (Pin_1)
- net at J1.C12: now also D?.1 (Pin_1)
- net at J1.C13: now also D?.1 (Pin_1)
- net at J1.C14: now also D?.1 (Pin_1)
- net at J1.C15: now also D?.1 (Pin_1)
- net at J1.C17: now also D?.1 (Pin_1)
- net at J1.C18: now also D?.1 (Pin_1)
- net at J1.C19: now also D?.1 (Pin_1)
- net at J1.C2: now also D?.1 (Pin_1)
- net at J1.C20: now also D?.1 (Pin_1)
- net at J1.C3: now also D?.1 (Pin_1)
- net at J1.C4: now also D?.1 (Pin_1)
- net at J1.C6: now also D?.1 (Pin_1)
- net at J1.C7: now also D?.1 (Pin_1)
- net at J1.C9: now also D?.1 (Pin_1)
- net at J1.B10: now also ALTL.1 (Pin_1)
- net at J1.B13: now also ALTF.1 (Pin_1)
- net OUT_MCS: now reaches J1.B15
- net OUT_MCS: now also D?.2 (A)
- net at J1.B18: now also ALTC.1 (Pin_1)
- net at J1.B19: now also SEFD.1 (Pin_1)
- net at J1.B20: now also SEDF.1 (Pin_1)
- net OUT_PURGE: now reaches J1.B21
- net OUT_INJ3: now reaches J1.B3
- net OUT_INJ1: now reaches J1.B5
- net at J1.D10: now also D?.1 (Pin_1)
- net at J1.D12: now also D?.1 (Pin_1)
- net at J1.D15: now also D?.1 (Pin_1)
- net at J1.D2: now also D2.1 (Pin_1)
- net at J1.D3: now also D3.1 (Pin_1)
- net at J1.D5: now also ATPR.1 (Pin_1)
- net at J1.D6: now also ATPP.1 (Pin_1)
- net at J1.D9: now also D?.1 (Pin_1)
- net at J1.E12: now also D?.1 (Pin_1)
- net at J1.E13: now also D?.1 (Pin_1)
- net IN_FTPS: now reaches J1.E14
- net at J1.E15: now also D?.1 (Pin_1)
- net at J1.E16: now also D?.1 (Pin_1)
- net OUT_MAIN2: now reaches J1.E17
- net at J1.E18: now also D?.1 (Pin_1)
- net OUT_VENT: now reaches J1.E19
- net at J1.E2: now also D?.1 (Pin_1)
- net at J1.E20: now also D?.1 (Pin_1)
- net at J1.E21: now also D?.1 (Pin_1)
- net IN_BRAKE: now reaches J1.E22
- net at J1.E23: now also D?.1 (Pin_1)
- net at J1.E25: now also D?.1 (Pin_1)
- net at J1.E26: now also D?.1 (Pin_1)
- net at J1.E27: now also D?.1 (Pin_1)
- net at J1.E29: now also D?.1 (Pin_1)
- net at J1.E3: now also D?.1 (Pin_1)
- net at J1.E30: now also D?.1 (Pin_1)
- net OUT_CHECK_ENGINE: now reaches J1.E31
- net OUT_MAIN: now reaches J1.E7
- net OUT_MAF_RELAY: now reaches J1.E8
- net IN_VIGN: now reaches J1.E9
- new net: M?.V2 (CAN_VIO), M?.W2 (CAN_VIO)
- new net: M?.V6 (CAN_RX), M?.W3 (CAN_RX)
- new net: M?.V5 (CAN_TX), M?.W4 (CAN_TX)
- new net: J?.5 (Pin_5), M?.W5 (nReset)
- new net: J?.4 (Pin_4), M?.W6 (SWDIO)
- new net: J?.2 (Pin_2), M?.W7 (SWCLK)
- new net: J?.1 (Pin_1), M?.W8 (V33_OUT)
- no-connect marks 0 -> 31
Other:
- note added: "ETB Relay"
- note added: "MAF HEAT?"
- note added: "MAF?"
- note added: "MR???"
- note added: "PSP???"
- moved on the sheet: J2, J3, J4

Commit message: Upd pinout
Parts:
- removed ALTC, ALTF, ALTL, ATPP, ATPR, D3, D? (x19), SEDF, SEFD: Pad, hellen-one-common:PAD-TH, symbol hellen-one-common:Pad
- removed D2, D? (x17): S-MODE, hellen-one-common:PAD-TH, symbol hellen-one-common:Pad
- added P? (x50): Pad, hellen-one-common:PAD-TH, symbol hellen-one-common:Pad
- renumbered J3 to J?, J1 to J?, J2 to J?, J4 to J?
Connections:
- net IN_BRAKE is gone; now on net AV5: J?.E22
- net IN_VIGN is gone; now on net 12V_RAW: J?.E9
- net OUT_CHECK_ENGINE is gone; now on net LS6: J?.E31
- net OUT_INJ1 is gone; now on net LS4: J?.B5
- net OUT_INJ3 is gone; now on net LS2: J?.B3
- net OUT_MAIN is gone; now on net LS5: J?.E7
- net CAN+: now also J?.E11
- net CAN-: now also J?.E24
- net at J?.E20: now also P?.1 (Pin_1)
- net at J?.D2: now also P?.1 (Pin_1)
- net at J?.E25: now also P?.1 (Pin_1)
- net at J?.C2: now also P?.1 (Pin_1)
- net at J?.D3: now also P?.1 (Pin_1)
- net at J?.B13: now also P?.1 (Pin_1)
- net at J?.E21: now also P?.1 (Pin_1)
- net at J?.D15: now also P?.1 (Pin_1)
- net at J?.E12: now also P?.1 (Pin_1)
- net at J?.C1: now also P?.1 (Pin_1)
- net at J?.C10: now also P?.1 (Pin_1)
- net at J?.C11: now also P?.1 (Pin_1)
- net at J?.C12: now also P?.1 (Pin_1)
- net at J?.C13: now also P?.1 (Pin_1)
- net at J?.C14: now also P?.1 (Pin_1)
- net at J?.C15: now also P?.1 (Pin_1)
- net at J?.C17: now also P?.1 (Pin_1)
- net at J?.C18: now also P?.1 (Pin_1)
- net at J?.C19: now also P?.1 (Pin_1)
- net at J?.C20: now also P?.1 (Pin_1)
- net at J?.C21: now also P?.1 (Pin_1)
- net at J?.C22: now also P?.1 (Pin_1)
- net at J?.C3: now also P?.1 (Pin_1)
- net at J?.C4: now also P?.1 (Pin_1)
- net at J?.C5: now also P?.1 (Pin_1)
- net at J?.C6: now also P?.1 (Pin_1)
- net at J?.C7: now also P?.1 (Pin_1)
- net at J?.C9: now also P?.1 (Pin_1)
- net at J?.E13: now also P?.1 (Pin_1)
- net at J?.E15: now also P?.1 (Pin_1)
- net at J?.B10: now also P?.1 (Pin_1)
- net at J?.B18: now also P?.1 (Pin_1)
- net at J?.B19: now also P?.1 (Pin_1)
- net at J?.B20: now also P?.1 (Pin_1)
- net at J?.E16: now also P?.1 (Pin_1)
- net at J?.E30: now also P?.1 (Pin_1)
- net at J?.D6: now also P?.1 (Pin_1)
- net at J?.D5: now also P?.1 (Pin_1)
- net at J?.E2: now also P?.1 (Pin_1)
- net at J?.E26: now also P?.1 (Pin_1)
- net at J?.E29: now also P?.1 (Pin_1)
- net at J?.D9: now also P?.1 (Pin_1)
- net at J?.D12: now also P?.1 (Pin_1)
- net at J?.E23: now also P?.1 (Pin_1)
- net at J?.E27: now also P?.1 (Pin_1)
- net at J?.E3: now also P?.1 (Pin_1)
- net at J?.E18: now also P?.1 (Pin_1)
- net at J?.D10: now also P?.1 (Pin_1)
- net at J?.D8: now also P?.1 (Pin_1)
- net at J?.E1: now also P?.1 (Pin_1)
- no-connect marks 31 -> 24
Other:
- note added: "AT"
- note added: "Do we need this?"
- note added: "ETB Relay???"
- note removed: "ETB Relay"
- note removed: "MR???"

Commit message: Upd pinout
Parts:
- added F1, F2: Fuse-Pad-Pad, hellen-one-common:PAD-1206-PAD, symbol hellen-one-common:Fuse-Pad-Pad
- added J2: XH-8A, hellen-one-common:XH-8A, symbol Connector_Generic:Conn_01x08
- added P1, P16, P2, P24, P3, P56, P57, P58, P59, P60, P61, P62, P63, P64, P65, P66, P67, P68, P69, P70, P71, P72, P73, P74, P75, P76, P77, P78, P79, P80, P81, P82, P83, P84, P85, P86, P87, P88, P? (x9): Pad, hellen-one-common:PAD-TH, symbol hellen-one-common:Pad
- gave numbers to parts that had none: 58
Connections:
- net OUT_MAIN2 is gone; now on net LS9: J1.E17
- net 12V_MR: now also F1.2, F2.2; no longer J1.A2, J1.A3
- net 5V_SENSOR_1: now also P57.1 (Pin_1)
- net 5V_SENSOR_2: now also M1.W1 (V5_IN), M2.V1 (V5), P58.1 (Pin_1)
- net AT3: now also P60.1 (Pin_1)
- net AT4: now also P56.1 (Pin_1)
- net AV10: now also P77.1 (Pin_1)
- net AV11: now also P75.1 (Pin_1)
- net AV6: now also P?.1 (Pin_1)
- net AV7: now also J1.A30
- net AV8: now also P76.1 (Pin_1)
- net AV9: now also P74.1 (Pin_1)
- net CAN+: now also M2.S2 (CANH)
- net CAN-: now also M2.S1 (CANL)
- net CAN2+: now also P88.1 (Pin_1)
- net CAN2-: now also P87.1 (Pin_1)
- net DIGITAL_6: now also P83.1 (Pin_1)
- net ETB1+: now also P81.1 (Pin_1)
- net ETB1-: now also P80.1 (Pin_1)
- net ETB2+: now also P86.1 (Pin_1)
- net ETB2-: now also P82.1 (Pin_1)
- net GND: now also M1.E6 (LSU_H-), M1.G (GND), M2.E1 (GND), J2.1 (Pin_1), J2.2 (Pin_2)
- net HS1: now also P62.1 (Pin_1)
- net HS2: now also P61.1 (Pin_1)
- net HS3: now also P64.1 (Pin_1)
- net HS4: now also P65.1 (Pin_1)
- net IGN10: now also P68.1 (Pin_1)
- net IGN11: now also P67.1 (Pin_1)
- net IGN12: now also P66.1 (Pin_1)
- net IGN5: now also P73.1 (Pin_1)
- net IGN6: now also P72.1 (Pin_1)
- net IGN7: now also P71.1 (Pin_1)
- net IGN8: now also P70.1 (Pin_1)
- net IGN9: now also P69.1 (Pin_1)
- net KNOCK_2: now also P59.1 (Pin_1)
- net LS10: now also P?.1 (Pin_1)
- net LS11: now also P63.1 (Pin_1)
- net LS12: now also P?.1 (Pin_1)
- net LS7: now also P?.1 (Pin_1)
- net LS8: now also P?.1 (Pin_1)
- net VR1+: now also P79.1 (Pin_1)
- net VR1-: now also P85.1 (Pin_1)
- net VR2+: now also P78.1 (Pin_1)
- net VR2-: now also P84.1 (Pin_1)
- net at J1.A10: now also P1.1 (Pin_1)
- net at J1.A28: now also P2.1 (Pin_1)
- net at J1.A31: now also P3.1 (Pin_1)
- net WBO_Vs: now reaches M1.E1 (LSU_Un)
- net WBO_Vs: now also J2.8 (Pin_8)
- net WBO_Vs/Ip: now reaches M1.E2 (LSU_Vm)
- net WBO_Vs/Ip: now also J2.7 (Pin_7)
- net WBO_Ip: now reaches M1.E3 (LSU_Ip)
- net WBO_Ip: now also J2.6 (Pin_6)
- net WBO_R_Trim: now reaches M1.E4 (LSU_Rtrim)
- net WBO_R_Trim: now also J2.5 (Pin_5)
- net WBO_H-: now reaches M1.E5 (LSU_H+)
- net WBO_H-: now also J2.3 (Pin_3), J2.4 (Pin_4)
- net at M1.J1 (SEL1): now also M1.J_GND1 (PULL_DOWN1)
- net at J1.C16: now also P24.1 (Pin_1)
- net at J1.C8: now also P16.1 (Pin_1)
- net IN_FTPS: no longer names the net of J1.E14
- net IN_FTPS: now also P?.1 (Pin_1)
- net OUT_MAF_RELAY: no longer names the net of J1.E8
- net OUT_MAF_RELAY: now also P?.1 (Pin_1)
- net OUT_PURGE: no longer names the net of J1.B21
- net OUT_PURGE: now also P?.1 (Pin_1)
- net OUT_VENT: no longer names the net of J1.E19
- net OUT_VENT: now also P?.1 (Pin_1)
- new net: F1.1, J1.A2
- new net: F2.1, J1.A3
- no-connect marks 24 -> 26
Other:
- note added: "#0"
- note removed: "Do we need this?"
- note removed: "MAF HEAT?"
- note removed: "MAF?"
- note removed: "PSP???"

Commit message: Upd pcb
Parts:
- added J10, J11, J12, J13, J7, J8, J9: Conn_01x01, MountingHole:MountingHole_4.5mm, symbol Connector_Generic:Conn_01x01
- gave numbers to parts that had none: 9

Commit message: Proteus-compatible component
Parts:
- removed J1: 1318612-1, lib:13186121, symbol 1318612-1:1318612-1
- added D2: proteus, kicad6-libraries:proteus, symbol proteus:proteus
- added G1, G2, G3, G4, G5: PROTO_AREA, hellen-one-common:PROTO_AREA, symbol hellen-one-common:PROTO_AREA
- added J1: 1318612-1, kicad6-libraries:TE_1318612-1, symbol TE_1318612-1:1318612-1
Connections:
- net 12V_PROT: now also G5.11, G5.12, G5.13, G5.14, G5.15
- net 12V_RAW: now also J1.E9
- net 5V_SENSOR_1: now also J1.A20, J1.A21, J1.E5
- net 5V_SENSOR_2: now also G5.10, G5.6, G5.7, G5.8, G5.9
- net AT1: now also J1.B17
- net AT2: now also J1.B8
- net AV1: now also J1.A25
- net AV2: now also J1.A26
- net AV3: now also J1.A29
- net AV4: now also J1.B22
- net AV5: now also J1.E22
- net AV7: now also J1.A30
- net CAN+: now also J1.E11
- net CAN-: now also J1.E24
- net DIGITAL_1: now also J1.A6
- net DIGITAL_2: now also J1.A7
- net DIGITAL_3: now also J1.A18
- net DIGITAL_4: now also J1.A19
- net DIGITAL_5: now also J1.B11
- net GND: now also G5.1, G5.2, G5.3, G5.4, G5.5, J1.A23, J1.A24, J1.A4, J1.A5, J1.A8, J1.A9, J1.E4
- net IGN1: now also J1.A16
- net IGN2: now also J1.A15
- net IGN3: now also J1.A14
- net IGN4: now also J1.A13
- net IN_KNOCK: now also J1.A1
- net LS1: now also J1.B2
- net LS13: now also J1.A12
- net LS14: now also J1.A11
- net LS15: now also J1.B1
- net LS16: now also J1.B6
- net LS2: now also J1.B3
- net LS3: now also J1.B4
- net LS4: now also J1.B5
- net LS5: now also J1.E7
- net LS6: now also J1.E31
- net LS9: now also J1.E17
- net OUT_MCS: now also J1.B15
- net at P34.1 (Pin_1): now also J1.D6
- net at P52.1 (Pin_1): now also J1.E26
- net at P22.1 (Pin_1): now also J1.C14
- net at P32.1 (Pin_1): now also J1.D3
- net at P16.1 (Pin_1): now also J1.C8
- net at P55.1 (Pin_1): now also J1.E30
- net at P39.1 (Pin_1): now also J1.D15
- net at P7.1 (Pin_1): now also J1.B19
- net at P49.1 (Pin_1): now also J1.E21
- net at P1.1 (Pin_1): now also J1.A10
- net at F1.1: now also J1.A2
- net at P2.1 (Pin_1): now also J1.A28
- net at F2.1: now also J1.A3
- net at P3.1 (Pin_1): now also J1.A31
- net at P50.1 (Pin_1): now also J1.E23
- net at P10.1 (Pin_1): now also J1.C2
- net at P43.1 (Pin_1): now also J1.E12
- net at P23.1 (Pin_1): now also J1.C15
- net at P33.1 (Pin_1): now also J1.D5
- net at P41.1 (Pin_1): now also J1.E2
- net at P47.1 (Pin_1): now also J1.E18
- net at P12.1 (Pin_1): now also J1.C4
- net at P9.1 (Pin_1): now also J1.C1
- net at P18.1 (Pin_1): now also J1.C10
- net at P19.1 (Pin_1): now also J1.C11
- net at P20.1 (Pin_1): now also J1.C12
- net at P21.1 (Pin_1): now also J1.C13
- net at P24.1 (Pin_1): now also J1.C16
- net at P25.1 (Pin_1): now also J1.C17
- net at P26.1 (Pin_1): now also J1.C18
- net at P27.1 (Pin_1): now also J1.C19
- net at P28.1 (Pin_1): now also J1.C20
- net at P29.1 (Pin_1): now also J1.C21
- net at P30.1 (Pin_1): now also J1.C22
- net at P11.1 (Pin_1): now also J1.C3
- net at P13.1 (Pin_1): now also J1.C5
- net at P14.1 (Pin_1): now also J1.C6
- net at P15.1 (Pin_1): now also J1.C7
- net at P17.1 (Pin_1): now also J1.C9
- net at P90.1 (Pin_1): now also J1.E8
- net at P36.1 (Pin_1): now also J1.D9
- net at P4.1 (Pin_1): now also J1.B10
- net at P5.1 (Pin_1): now also J1.B13
- net at P6.1 (Pin_1): now also J1.B18
- net at P8.1 (Pin_1): now also J1.B20
- net at P89.1 (Pin_1): now also J1.B21
- net at P38.1 (Pin_1): now also J1.D12
- net at P91.1 (Pin_1): now also J1.E14
- net at P44.1 (Pin_1): now also J1.E13
- net at P92.1 (Pin_1): now also J1.E19
- net at P48.1 (Pin_1): now also J1.E20
- net at P40.1 (Pin_1): now also J1.E1
- net at P53.1 (Pin_1): now also J1.E27
- net at P37.1 (Pin_1): now also J1.D10
- net at P46.1 (Pin_1): now also J1.E16
- net at P54.1 (Pin_1): now also J1.E29
- net at P45.1 (Pin_1): now also J1.E15
- net at P51.1 (Pin_1): now also J1.E25
- net at P35.1 (Pin_1): now also J1.D8
- net at P31.1 (Pin_1): now also J1.D2
- net at P42.1 (Pin_1): now also J1.E3
- new net: G2.1, G2.11, G2.6
- new net: G2.10, G2.15, G2.5
- new net: G2.12, G2.2, G2.7
- new net: G2.13, G2.3, G2.8
- new net: G2.14, G2.4, G2.9
- new net: G3.1, G3.11, G3.6
- new net: G3.10, G3.15, G3.5
- new net: G3.12, G3.2, G3.7
- new net: G3.13, G3.3, G3.8
- new net: G3.14, G3.4, G3.9
- new net: G4.1, G4.11, G4.6
- new net: G4.10, G4.15, G4.5
- new net: G4.12, G4.2, G4.7
- new net: G4.13, G4.3, G4.8
- new net: G4.14, G4.4, G4.9
- new net: G1.1, G1.11, G1.6
- new net: G1.10, G1.15, G1.5
- new net: G1.12, G1.2, G1.7
- new net: G1.13, G1.3, G1.8
- new net: G1.14, G1.4, G1.9
Other:
- moved on the sheet: J4, J5, J6, P56, P57, P58, P59, P60, P61, P62, P63, P64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

Commit message: Proteus-compatible board preview
Parts:
- removed J4: Conn_01x35, lib:ampseal-35, symbol Connector_Generic:Conn_01x35
- removed J5: Conn_01x35, lib:ampseal-35-2, symbol Connector_Generic:Conn_01x35
- removed J6: Conn_01x23, lib:ampseal-23, symbol Connector_Generic:Conn_01x23
- removed M1: Module-wbo-0.2, hellen-one-wbo-0.2:wbo, symbol hellen-one-wbo-0.2:Module-wbo-0.2
- removed P64, P97: Pad, hellen-one-common:PAD-TH, symbol hellen-one-common:Pad
- added F3: Fuse-Pad-Pad, hellen-one-common:PAD-1206-PAD, symbol hellen-one-common:Fuse-Pad-Pad
- added G6: RUSEFI_LOGO, kicad6-libraries:rusefi_logo, symbol rusefi_logo:RUSEFI_LOGO
- added G7, G8: PROTO_AREA, hellen-one-common:PROTO_AREA, symbol hellen-one-common:PROTO_AREA
- added M1: Module-wbo-0.3, hellen-one-wbo-0.3:wbo, symbol hellen-one-wbo-0.3:Module-wbo-0.3
- renumbered D2 to BRD1
Connections:
- net AT1 is gone; now on net IN_IAT: J1.B17
- net AT2 is gone; now on net IN_CLT: J1.B8
- net AT3 is gone; now on an unnamed net: P60.1 (Pin_1)
- net AT4 is gone; now on an unnamed net: P56.1 (Pin_1)
- net AV1 is gone; now on net IN_PPS2: J1.A25
- net AV10 is gone; now on an unnamed net: P77.1 (Pin_1)
- net AV11 is gone; now on an unnamed net: P75.1 (Pin_1)
- net AV2 is gone; now on net IN_PPS1: J1.A26
- net AV3 is gone; now on net IN_TPS: J1.A29
- net AV4 is gone; now on net IN_MRC: J1.B22
- net AV5 is gone; now on net IN_BRAKE: J1.E22
- net AV7 is gone; now on net IN_MAP: J1.A30
- net AV8 is gone; now on an unnamed net: P76.1 (Pin_1)
- net AV9 is gone; now on an unnamed net: P74.1 (Pin_1)
- net CAN+ is gone; now on net CAN_H: J1.E11, M2.S2 (CANH)
- net CAN- is gone; now on net CAN_L: J1.E24, M2.S1 (CANL)
- net CAN2+ is gone; now on an unnamed net: P88.1 (Pin_1)
- net CAN2- is gone; now on an unnamed net: P87.1 (Pin_1)
- net DIGITAL_1 is gone; now on net IN_CAM2: J1.A6
- net DIGITAL_2 is gone; now on net IN_CRANK: J1.A7
- net DIGITAL_3 is gone; now on net IN_VSS: J1.A18
- net DIGITAL_4 is gone; now on net IN_CAM1: J1.A19
- net DIGITAL_5 is gone; now on net IN_VTPSW: J1.B11
- net DIGITAL_6 is gone; now on an unnamed net: P83.1 (Pin_1)
- net ETB1+ is gone; now on an unnamed net: P81.1 (Pin_1)
- net ETB1- is gone; now on an unnamed net: P80.1 (Pin_1)
- net ETB2+ is gone; now on an unnamed net: P86.1 (Pin_1)
- net ETB2- is gone; now on an unnamed net: P82.1 (Pin_1)
- net HS1 is gone; now on an unnamed net: P62.1 (Pin_1)
- net HS2 is gone; now on an unnamed net: P61.1 (Pin_1)
- net HS4 is gone; now on an unnamed net: P65.1 (Pin_1)
- net IGN1 is gone; now on net OUT_IGN1: J1.A16
- net IGN10 is gone; now on an unnamed net: P68.1 (Pin_1)
- net IGN11 is gone; now on an unnamed net: P67.1 (Pin_1)
- net IGN12 is gone; now on an unnamed net: P66.1 (Pin_1)
- net IGN2 is gone; now on net OUT_IGN2: J1.A15
- net IGN3 is gone; now on net OUT_IGN3: J1.A14
- net IGN4 is gone; now on net OUT_IGN4: J1.A13
- net IGN5 is gone; now on an unnamed net: P73.1 (Pin_1)
- net IGN6 is gone; now on an unnamed net: P72.1 (Pin_1)
- net IGN7 is gone; now on an unnamed net: P71.1 (Pin_1)
- net IGN8 is gone; now on an unnamed net: P70.1 (Pin_1)
- net IGN9 is gone; now on an unnamed net: P69.1 (Pin_1)
- net KNOCK_2 is gone; now on an unnamed net: P59.1 (Pin_1)
- net LS1 is gone; now on net OUT_INJ4: J1.B2
- net LS10 is gone; now on an unnamed net: P95.1 (Pin_1)
- net LS11 is gone; now on an unnamed net: P63.1 (Pin_1)
- net LS12 is gone; now on an unnamed net: P96.1 (Pin_1)
- net LS13 is gone; now on net OUT_IAC: J1.A12
- net LS14 is gone; now on net OUT_IMRC: J1.A11
- net LS15 is gone; now on net OUT_VTC: J1.B1
- net LS16 is gone; now on net OUT_VTS: J1.B6
- net LS2 is gone; now on net OUT_INJ3: J1.B3
- net LS3 is gone; now on net OUT_INJ2: J1.B4
- net LS4 is gone; now on net OUT_INJ1: J1.B5
- net LS5 is gone; now on net OUT_MAIN: J1.E7
- net LS6 is gone; now on net OUT_CHECK_ENGINE: J1.E31
- net LS7 is gone; now on an unnamed net: P93.1 (Pin_1)
- net LS8 is gone; now on an unnamed net: P94.1 (Pin_1)
- net LS9 is gone; now on net OUT_FUEL_PUMP: J1.E17
- net VR1+ is gone; now on an unnamed net: P79.1 (Pin_1)
- net VR1- is gone; now on an unnamed net: P85.1 (Pin_1)
- net VR2+ is gone; now on an unnamed net: P78.1 (Pin_1)
- net VR2- is gone; now on an unnamed net: P84.1 (Pin_1)
- net 12V_MR: now also BRD1.B23 (12V_MR)
- net 12V_PROT: now also BRD1.C11 (12V_PROT), BRD1.C12 (12V_PROT)
- net 5V_SENSOR_1: now also BRD1.C21 (5V_1), BRD1.C32 (5V_1), BRD1.C9 (5V_1); no longer P57.1 (Pin_1)
- net 5V_SENSOR_2: now also BRD1.C10 (5V_2), BRD1.C22 (5V_2), BRD1.C33 (5V_2), M1.W1 (V5_IN); no longer P58.1 (Pin_1)
- net GND: now also BRD1.A17 (GND), BRD1.A18 (GND), BRD1.A24 (GND), BRD1.B19 (GND), BRD1.B20 (GND), BRD1.C1 (GND_SENS), BRD1.C2 (GND_SENS), BRD1.C23 (GND_SENS), BRD1.C29 (GND_SENS), BRD1.C3 (GND_SENS), BRD1.C4 (GND_SENS), BRD1.C5 (GND_SENS), BRD1.C6 (GND_SENS), BRD1.C7 (GND_SENS), BRD1.C8 (GND_SENS), M1.E6 (LSU_H-), M1.G (GND)
- net IN_KNOCK: now also BRD1.C34 (KNOCK1)
- net OUT_MCS: now also BRD1.A21 (LS12)
- net WBO_H-: now also M1.E5 (LSU_H+)
- net WBO_Ip: now also M1.E3 (LSU_Ip)
- net WBO_R_Trim: now also M1.E4 (LSU_Rtrim)
- net WBO_Vs: now also M1.E1 (LSU_Un)
- net WBO_Vs/Ip: now also M1.E2 (LSU_Vm)
- net at M2.V2 (CAN_VIO): now also M1.W2 (CAN_VIO)
- net at M2.V6 (CAN_RX): now also M1.W3 (CAN_RX)
- net at M2.V5 (CAN_TX): now also M1.W4 (CAN_TX)
- net at J3.5 (Pin_5): now also M1.W5 (nReset)
- net at J3.4 (Pin_4): now also M1.W6 (SWDIO)
- net at J3.2 (Pin_2): now also M1.W7 (SWCLK)
- net at J3.1 (Pin_1): now also M1.W8 (V33_OUT)
- net at BRD1.A1 (HS2): now also P57.1 (Pin_1)
- net OUT_IAC: now reaches BRD1.A10 (LS13)
- net OUT_IMRC: now reaches BRD1.A11 (LS14)
- net OUT_VTS: now reaches BRD1.A12 (LS15)
- net at BRD1.A13 (HS3): now also P58.1 (Pin_1)
- net OUT_INJ1: now reaches BRD1.A19 (LS8)
- net OUT_CHECK_ENGINE: now reaches BRD1.A20 (LS10)
- net OUT_IGN3: now reaches BRD1.A22 (IGN3)
- net OUT_VTC: now reaches BRD1.A23 (LS16)
- net OUT_IGN4: now reaches BRD1.A33 (IGN4)
- net OUT_IGN2: now reaches BRD1.A34 (IGN2)
- net OUT_IGN1: now reaches BRD1.A35 (IGN1)
- net OUT_INJ4: now reaches BRD1.A5 (LS5)
- net OUT_INJ3: now reaches BRD1.A6 (LS6)
- net OUT_INJ2: now reaches BRD1.A7 (LS7)
- net OUT_MAIN: now reaches BRD1.A8 (LS9)
- net OUT_FUEL_PUMP: now reaches BRD1.A9 (LS11)
- net IN_CRANK: now reaches BRD1.B1 (D2)
- net IN_CAM2: now reaches BRD1.B10 (D1)
- net CAN_L: now reaches BRD1.B16 (CAN-)
- net CAN_H: now reaches BRD1.B17 (CAN+)
- net IN_VIGN: now reaches BRD1.B18 (12V_IGN)
- net IN_VIGN: now also F3.2
- net IN_VSS: now reaches BRD1.B2 (D3)
- net IN_CAM1: now reaches BRD1.B3 (D4)
- net IN_VTPSW: now reaches BRD1.B9 (D5)
- net IN_PPS2: now reaches BRD1.C13 (AV1)
- net IN_TPS: now reaches BRD1.C14 (AV3)
- net IN_BRAKE: now reaches BRD1.C15 (AV5)
- net IN_IAT: now reaches BRD1.C19 (AT1)
- net IN_PPS1: now reaches BRD1.C24 (AV2)
- net IN_MRC: now reaches BRD1.C25 (AV4)
- net IN_MAP: now reaches BRD1.C26 (AV6)
- net IN_CLT: now reaches BRD1.C30 (AT2)
- net 12V_RAW: no longer names the net of J1.E9
- net 12V_RAW: now also F3.1
- new net: G8.1, G8.11, G8.6
- new net: G8.10, G8.15, G8.5
- new net: G8.12, G8.2, G8.7
- new net: G8.13, G8.3, G8.8
- new net: G8.14, G8.4, G8.9
- new net: M1.J1 (SEL1), M1.J_GND1 (PULL_DOWN1)
- new net: G7.1, G7.11, G7.6
- new net: G7.10, G7.15, G7.5
- new net: G7.12, G7.2, G7.7
- new net: G7.13, G7.3, G7.8
- new net: G7.14, G7.4, G7.9
Other:
- note removed: "BLACK"
- note removed: "WHITE"
- moved on the sheet: BRD1
