File: proteus125honda.kicad_sch (KiCad schematic)
At the start: 120 parts, among them J1 1318612-1, J10 Conn_01x01, J11 Conn_01x01, J12 Conn_01x01, J13 Conn_01x01, J2 XH-8A, J3 Conn_01x06, J7 Conn_01x01, J8 Conn_01x01, J9 Conn_01x01, M1 Module-wbo-0.3, M2 Module-can-0.1, P1 Pad, P10 Pad, P11 Pad, P12 Pad, P13 Pad, P14 Pad, P15 Pad, P16 Pad, P17 Pad, P18 Pad, P19 Pad, P2 Pad, P20 Pad, P21 Pad, P22 Pad, P23 Pad, P24 Pad, P25 Pad, P26 Pad, P27 Pad, P28 Pad, P29 Pad, P3 Pad, P30 Pad, P31 Pad, P32 Pad, P33 Pad, P34 Pad, P35 Pad, P36 Pad, P37 Pad, P38 Pad, P39 Pad, P4 Pad, P40 Pad, P41 Pad, P42 Pad, P43 Pad, P44 Pad, P45 Pad, P46 Pad, P47 Pad, P48 Pad, P49 Pad, P5 Pad, P50 Pad, P51 Pad, P52 Pad, P53 Pad, P54 Pad, P55 Pad, P56 Pad, P57 Pad, P58 Pad, P59 Pad, P6 Pad, P60 Pad, P61 Pad, P62 Pad, P63 Pad, P65 Pad, P66 Pad, P67 Pad, P68 Pad, P69 Pad, P7 Pad, P70 Pad, P71 Pad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

Commit message: MAP
Parts:
- removed P85: Pad, hellen-one-common:PAD-TH, symbol hellen-one-common:Pad
- added C1: 100n, hellen-one-common:C0603, symbol hellen-one-common:Cap
- added C2: 47p, hellen-one-common:C0603, symbol hellen-one-common:Cap
- added R1: 51k, hellen-one-common:R0603, symbol hellen-one-common:Res
- added U1: MPXxx6115A, kicad6-libraries:MPX_SOP_SSOP, symbol MPX_SOP_SSOP:MPXxx6115A
Connections:
- net 5V_SENSOR_2: now also C1.2, U1.2 (Vs)
- net GND: now also C1.1, C2.1, R1.2, U1.3 (GND)
- net at BRD1.C16 (AV7): now also C2.2, R1.1, U1.4 (Vout)
Changed lines of the file:
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@@
   (junction (at 165.1 392.43) (diameter 0) (color 0 0 0 0))
   (junction (at 165.1 398.78) (diameter 0) (color 0 0 0 0))
+  (junction (at 167.64 267.97) (diameter 0) (color 0 0 0 0))
+  (junction (at 167.64 275.59) (diameter 0) (color 0 0 0 0))
+  (junction (at 207.01 267.97) (diameter 0) (color 0 0 0 0))
+  (junction (at 210.82 278.13) (diameter 0) (color 0 0 0 0))
+  (junction (at 213.36 267.97) (diameter 0) (color 0 0 0 0))
   (junction (at 267.97 242.57) (diameter 1.016) (color 0 0 0 0))
   (junction (at 269.24 160.02) (diameter 0) (color 0 0 0 0))
@@
     (stroke (width 0) (type default) (color 0 0 0 0))
   )
+  (wire (pts (xy 162.56 267.97) (xy 167.64 267.97))
+    (stroke (width 0) (type default) (color 0 0 0 0))
+  )
   (wire (pts (xy 165.1 373.38) (xy 168.91 373.38))
     (stroke (width 0) (type default) (color 0 0 0 0))
@@
     (stroke (width 0) (type default) (color 0 0 0 0))
   )
+  (wire (pts (xy 167.64 267.97) (xy 175.26 267.97))
+    (stroke (width 0) (type default) (color 0 0 0 0))
+  )
+  (wire (pts (xy 167.64 275.59) (xy 175.26 275.59))
+    (stroke (width 0) (type default) (color 0 0 0 0))
+  )
   (wire (pts (xy 175.26 26.67) (xy 186.69 26.67))
     (stroke (width 0) (type solid) (color 0 0 0 0))
@@
     (stroke (width 0) (type default) (color 0 0 0 0))
   )
+  (wire (pts (xy 198.12 267.97) (xy 207.01 267.97))
+    (stroke (width 0) (type default) (color 0 0 0 0))
+  )
+  (wire (pts (xy 207.01 267.97) (xy 213.36 267.97))
+    (stroke (width 0) (type default) (color 0 0 0 0))
+  )
+  (wire (pts (xy 207.01 278.13) (xy 207.01 275.59))
+    (stroke (width 0) (type default) (color 0 0 0 0))
+  )
+  (wire (pts (xy 210.82 278.13) (xy 207.01 278.13))
+    (stroke (width 0) (type default) (color 0 0 0 0))
+  )
+  (wire (pts (xy 210.82 278.13) (xy 213.36 278.13))
+    (stroke (width 0) (type default) (color 0 0 0 0))
+  )
+  (wire (pts (xy 213.36 267.97) (xy 269.24 267.97))
+    (stroke (width 0) (type default) (color 0 0 0 0))
+  )
   (wire (pts (xy 229.87 24.13) (xy 241.3 24.13))
     (stroke (width 0) (type default) (color 0 0 0 0))
@@
     (effects (font (size 1.27 1.27)) (justify left bottom))
   )
+  (label "5V_SENSOR_2" (at 162.56 267.97 180)
+    (effects (font (size 1.27 1.27)) (justify right bottom))
+  )
   (label "5V_SENSOR_2" (at 184.15 21.59 180)
     (effects (font (size 1.27 1.27)) (justify right bottom))
@@
     (pin "1")
   )
+  (symbol (lib_id "power:GND") (at 167.64 275.59 0) (unit 1)
+    (in_bom yes) (on_board yes)
+    (property "Reference" "#PWR0101" (id 0) (at 167.64 281.94 0)
+      (effects (font (size 1.27 1.27)) hide)
+    )
+    (property "Value" "GND" (id 1) (at 169.6336 279.4268 0)
+      (effects (font (size 1.27 1.27)) (justify right))
+    )
+    (property "Footprint" "" (id 2) (at 167.64 275.59 0)
+      (effects (font (size 1.27 1.27)) hide)
+    )
+    (property "Datasheet" "" (id 3) (at 167.64 275.59 0)
+      (effects (font (size 1.27 1.27)) hide)
+    )
+    (pin "1")
+  )
   (symbol (lib_id "power:GND") (at 184.15 41.91 270) (mirror x) (unit 1)
     (in_bom yes) (on_board yes)
@@
     (pin "1")
   )
+  (symbol (lib_id "power:GND") (at 210.82 278.13 0) (unit 1)
+    (in_bom yes) (on_board yes)
+    (property "Reference" "#PWR0102" (id 0) (at 210.82 284.48 0)
+      (effects (font (size 1.27 1.27)) hide)
+    )
+    (property "Value" "GND" (id 1) (at 212.8136 281.9668 0)
+      (effects (font (size 1.27 1.27)) (justify right))
+    )
+    (property "Footprint" "" (id 2) (at 210.82 278.13 0)
+      (effects (font (size 1.27 1.27)) hide)
+    )
+    (property "Datasheet" "" (id 3) (at 210.82 278.13 0)
+      (effects (font (size 1.27 1.27)) hide)
+    )
+    (pin "1")
+  )
   (symbol (lib_id "power:GND") (at 229.87 31.75 0) (unit 1)
     (in_bom yes) (on_board yes)
@@
     (pin "1")
   )
-  (symbol (lib_id "hellen-one-common:Pad") (at 264.16 267.97 180) (unit 1)
-    (in_bom yes) (on_board yes)
-    (property "Reference" "P85" (id 0) (at 267.2715 266.7784 0))
-    (property "Value" "Pad" (id 1) (at 264.16 265.43 0)
-      (effects (font (size 1.27 1.27)) hide)
-    )
-    (property "Footprint" "hellen-one-common:PAD-TH" (id 2) (at 264.16 264.16 0)
-      (effects (font (size 1.27 1.27)) hide)
-    )
-    (property "Datasheet" "~" (id 3) (at 264.16 267.97 0)
-      (effects (font (size 1.27 1.27)) hide)
-    )
-    (pin "1")
-  )
   (symbol (lib_id "hellen-one-common:Pad") (at 264.16 270.51 180) (unit 1)
     (in_bom yes) (on_board yes)
@@
     (pin "2")
   )
+  (symbol (lib_id "hellen-one-common:Res") (at 213.36 267.97 270) (unit 1)
+    (in_bom yes) (on_board yes)
+    (property "Reference" "R1" (id 0) (at 216.9581 271.3701 90))
+    (property "Value" "51k" (id 1) (at 217.0199 273.9983 90))
+    (property "Footprint" "hellen-one-common:R0603" (id 2) (at 209.55 271.78 0)
+      (effects (font (size 1.27 1.27)) hide)
+    )
+    (property "Datasheet" "" (id 3) (at 213.36 267.97 0)
+      (effects (font (size 1.27 1.27)) hide)
+    )
+    (property "LCSC" "C23196" (id 4) (at 213.36 267.97 0)
+      (effects (font (size 1.27 1.27)) hide)
+    )
+    (pin "1")
+    (pin "2")
+  )
+  (symbol (lib_id "hellen-one-common:Cap") (at 167.64 271.78 270) (mirror x) (unit 1)
+    (in_bom yes) (on_board yes)
+    (property "Reference" "C1" (id 0) (at 164.8459 270.6306 90)
+      (effects (font (size 1.27 1.27)) (justify right))
+    )
+    (property "Value" "100n" (id 1) (at 164.8459 272.9293 90)
+      (effects (font (size 1.27 1.27)) (justify right))
+    )
+    (property "Footprint" "hellen-one-common:C0603" (id 2) (at 163.83 274.32 0)
+      (effects (font (size 1.27 1.27)) hide)
+    )
+    (property "Datasheet" "" (id 3) (at 167.64 275.59 90)
+      (effects (font (size 1.27 1.27)) hide)
+    )
+    (property "LCSC" "C14663" (id 4) (at 167.64 271.78 0)
+      (effects (font (size 1.27 1.27)) hide)
+    )
+    (pin "1")
+    (pin "2")
+  )
+  (symbol (lib_id "hellen-one-common:Cap") (at 207.01 271.78 270) (mirror x) (unit 1)
+    (in_bom yes) (on_board yes)
+    (property "Reference" "C2" (id 0) (at 204.2159 270.6306 90)
+      (effects (font (size 1.27 1.27)) (justify right))
+    )
+    (property "Value" "47p" (id 1) (at 204.2159 272.9293 90)
+      (effects (font (size 1.27 1.27)) (justify right))
+    )
+    (property "Footprint" "hellen-one-common:C0603" (id 2) (at 203.2 274.32 0)
+      (effects (font (size 1.27 1.27)) hide)
+    )
+    (property "Datasheet" "" (id 3) (at 207.01 275.59 90)
+      (effects (font (size 1.27 1.27)) hide)
+    )
+    (property "LCSC" "C1671" (id 4) (at 207.01 271.78 0)
+      (effects (font (size 1.27 1.27)) hide)
+    )
+    (pin "1")
+    (pin "2")
+  )
   (symbol (lib_id "rusefi_logo:RUSEFI_LOGO") (at 50.8 400.05 0) (unit 1)
     (in_bom yes) (on_board yes) (fields_autoplaced)
@@
     (pin "8")
   )
+  (symbol (lib_id "MPX_SOP_SSOP:MPXxx6115A") (at 180.34 265.43 0) (unit 1)
+    (in_bom yes) (on_board yes) (fields_autoplaced)
+    (property "Reference" "U1" (id 0) (at 186.69 261.5142 0))
+    (property "Value" "MPXxx6115A" (id 1) (at 186.69 264.2893 0))
+    (property "Footprint" "kicad6-libraries:MPX_SOP_SSOP" (id 2) (at 180.34 265.43 0)
+      (effects (font (size 1.27 1.27)) hide)
+    )
+    (property "Datasheet" "" (id 3) (at 180.34 265.43 0)
+      (effects (font (size 1.27 1.27)) hide)
+    )
+    (pin "1")
+    (pin "2")
+    (pin "3")
+    (pin "4")
+    (pin "5")
+    (pin "6")
+    (pin "7")
+    (pin "8")
+  )
   (symbol (lib_id "hellen-one-common:PROTO_AREA") (at 77.47 372.11 270) (unit 1)
     (in_bom yes) (on_board yes)
@@
       (reference "#PWR021") (unit 1) (value "GND") (footprint "")
     )
+    (path "/022656ed-b3ef-4642-b33f-e03a5c129cff"
+      (reference "#PWR0101") (unit 1) (value "GND") (footprint "")
+    )
+    (path "/7923f538-5985-40a0-9378-8ddacdcd40bb"
+      (reference "#PWR0102") (unit 1) (value "GND") (footprint "")
+    )
     (path "/d0500b2d-9ad9-4ab4-8526-8eaa6292993a"
       (reference "BRD1") (unit 1) (value "proteus") (footprint "kicad6-libraries:proteus")
     )
+    (path "/1d2f62ce-51e9-4708-a725-2841ee08b8b5"
+      (reference "C1") (unit 1) (value "100n") (footprint "hellen-one-common:C0603")
+    )
+    (path "/0835db08-a76b-4db8-bc18-68cb34796d32"
+      (reference "C2") (unit 1) (value "47p") (footprint "hellen-one-common:C0603")
+    )
     (path "/b48b19f9-eac5-4fe8-9824-7f9de0773dea"
       (reference "D1") (unit 1) (value "D_Schottky") (footprint "Diode_SMD:D_SMA")
@@
       (reference "P84") (unit 1) (value "Pad") (footprint "hellen-one-common:PAD-TH")
     )
-    (path "/cafb015e-ada5-4637-b1f8-433520c35cc7"
-      (reference "P85") (unit 1) (value "Pad") (footprint "hellen-one-common:PAD-TH")
-    )
     (path "/8053ffe7-fd05-4520-bc87-12d9a387bdc7"
       (reference "P86") (unit 1) (value "Pad") (footprint "hellen-one-common:PAD-TH")
@@
       (reference "P96") (unit 1) (value "Pad") (footprint "hellen-one-common:PAD-TH")
     )
+    (path "/4b69f5ca-b009-4b88-ae7b-721ead183b4f"
+      (reference "R1") (unit 1) (value "51k") (footprint "hellen-one-common:R0603")
+    )
+    (path "/56d42875-db96-4dcd-87bf-57d53391facd"
+      (reference "U1") (unit 1) (value "MPXxx6115A") (footprint "kicad6-libraries:MPX_SOP_SSOP")
+    )
   )

Commit message: Fix proteus
Parts:
- removed P84: Pad, hellen-one-common:PAD-TH, symbol hellen-one-common:Pad
Connections:
- net GND: now also BRD1.B14 (GND)
- net at P83.1 (Pin_1): now also BRD1.B21 (CAN2-); no longer BRD1.B22 (reserved)
- net at P82.1 (Pin_1): now also BRD1.B22 (CAN2+); no longer BRD1.B14 (reserved)
Changed lines of the file:
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@@
     (stroke (width 0) (type default) (color 0 0 0 0))
   )
-  (wire (pts (xy 257.81 234.95) (xy 269.24 234.95))
+  (wire (pts (xy 257.81 232.41) (xy 269.24 232.41))
     (stroke (width 0) (type default) (color 0 0 0 0))
   )
-  (wire (pts (xy 257.81 237.49) (xy 269.24 237.49))
+  (wire (pts (xy 257.81 234.95) (xy 269.24 234.95))
     (stroke (width 0) (type default) (color 0 0 0 0))
   )
@@
     (stroke (width 0) (type solid) (color 0 0 0 0))
   )
+  (wire (pts (xy 267.97 240.03) (xy 267.97 242.57))
+    (stroke (width 0) (type default) (color 0 0 0 0))
+  )
   (wire (pts (xy 267.97 242.57) (xy 267.97 245.11))
     (stroke (width 0) (type solid) (color 0 0 0 0))
@@
     (stroke (width 0) (type default) (color 0 0 0 0))
   )
+  (wire (pts (xy 269.24 240.03) (xy 267.97 240.03))
+    (stroke (width 0) (type default) (color 0 0 0 0))
+  )
   (wire (pts (xy 269.24 242.57) (xy 267.97 242.57))
     (stroke (width 0) (type solid) (color 0 0 0 0))
@@
     (effects (font (size 1.27 1.27)) (justify right bottom))
   )
-  (label "IN_VIGN" (at 257.81 234.95 180)
+  (label "IN_VIGN" (at 257.81 232.41 180)
     (effects (font (size 1.27 1.27)) (justify right bottom))
   )
-  (label "12V_MR" (at 257.81 237.49 180)
+  (label "12V_MR" (at 257.81 234.95 180)
     (effects (font (size 1.27 1.27)) (justify right bottom))
   )
@@
     (pin "1")
   )
-  (symbol (lib_id "hellen-one-common:Pad") (at 264.16 229.87 180) (unit 1)
-    (in_bom yes) (on_board yes)
-    (property "Reference" "P84" (id 0) (at 267.2715 228.6784 0))
-    (property "Value" "Pad" (id 1) (at 264.16 227.33 0)
-      (effects (font (size 1.27 1.27)) hide)
-    )
-    (property "Footprint" "hellen-one-common:PAD-TH" (id 2) (at 264.16 226.06 0)
-      (effects (font (size 1.27 1.27)) hide)
-    )
-    (property "Datasheet" "~" (id 3) (at 264.16 229.87 0)
-      (effects (font (size 1.27 1.27)) hide)
-    )
-    (pin "1")
-  )
   (symbol (lib_id "hellen-one-common:Pad") (at 264.16 270.51 180) (unit 1)
     (in_bom yes) (on_board yes)
@@
       (reference "P83") (unit 1) (value "Pad") (footprint "hellen-one-common:PAD-TH")
     )
-    (path "/d5aff035-4c78-44fc-ba29-fa541e8e01b6"
-      (reference "P84") (unit 1) (value "Pad") (footprint "hellen-one-common:PAD-TH")
-    )
     (path "/8053ffe7-fd05-4520-bc87-12d9a387bdc7"
