File: proteus125honda.kicad_sch (KiCad schematic)
At the start: 122 parts, among them J1 1318612-1, J10 Conn_01x01, J11 Conn_01x01, J12 Conn_01x01, J13 Conn_01x01, J2 XH-8A, J3 Conn_01x06, J7 Conn_01x01, J8 Conn_01x01, J9 Conn_01x01, M1 Module-wbo-0.3, M2 Module-can-0.1, P1 Pad, P10 Pad, P11 Pad, P12 Pad, P13 Pad, P14 Pad, P15 Pad, P16 Pad, P17 Pad, P18 Pad, P19 Pad, P2 Pad, P20 Pad, P21 Pad, P22 Pad, P23 Pad, P24 Pad, P25 Pad, P26 Pad, P27 Pad, P28 Pad, P29 Pad, P3 Pad, P30 Pad, P31 Pad, P32 Pad, P33 Pad, P34 Pad, P35 Pad, P36 Pad, P37 Pad, P38 Pad, P39 Pad, P4 Pad, P40 Pad, P41 Pad, P42 Pad, P43 Pad, P44 Pad, P45 Pad, P46 Pad, P47 Pad, P48 Pad, P49 Pad, P5 Pad, P50 Pad, P51 Pad, P52 Pad, P53 Pad, P54 Pad, P55 Pad, P56 Pad, P57 Pad, P58 Pad, P59 Pad, P6 Pad, P60 Pad, P61 Pad, P62 Pad, P63 Pad, P65 Pad, P66 Pad, P67 Pad, P68 Pad, P69 Pad, P7 Pad, P70 Pad, P71 Pad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

Commit message: Export
Parts:
- removed J2: XH-8A, hellen-one-common:XH-8A, symbol Connector_Generic:Conn_01x08
- removed P39, P4, P5, P59, P62, P63: Pad, hellen-one-common:PAD-TH, symbol hellen-one-common:Pad
- added J2: XH-10A, Connector_Molex:Molex_SPOX_5267-10A_1x10_P2.50mm_Vertical, symbol Connector_Generic:Conn_01x10
- added R2, R3: Jumper-Pad-Pad, hellen-one-common:PAD-0805-PAD, symbol hellen-one-common:Jumper-Pad-Pad
Connections:
- net 12V_MR: now also J2.10 (Pin_10), J2.9 (Pin_9)
- net GND: now also J2.1 (Pin_1), J2.2 (Pin_2)
- net OUT_IAC: now also BRD1.A12 (LS15); no longer BRD1.A10 (LS13)
- net OUT_IMRC: now also BRD1.A23 (LS16); no longer BRD1.A11 (LS14)
- net OUT_VTC: now also BRD1.A1 (HS2); no longer BRD1.A23 (LS16)
- net OUT_VTS: now also BRD1.A2 (HS1); no longer BRD1.A12 (LS15)
- net WBO_H-: now also J2.3 (Pin_3), J2.4 (Pin_4)
- net WBO_Ip: now also J2.6 (Pin_6)
- net WBO_R_Trim: now also J2.5 (Pin_5)
- net WBO_Vs: now also J2.8 (Pin_8)
- net WBO_Vs/Ip: now also J2.7 (Pin_7)
- net OUT_ETB_RELAY: now reaches J1.D15
- net OUT_ETB_RELAY: now also BRD1.A16 (LS4)
- net at P56.1 (Pin_1): now also BRD1.A10 (LS13); no longer BRD1.A2 (HS1)
- net at J1.B13: now also R3.1
- net at P57.1 (Pin_1): now also BRD1.A11 (LS14); no longer BRD1.A1 (HS2)
- net at J1.B10: now also R2.1
- net OUT_CHARGING_LIGHT: now reaches BRD1.A4 (LS3)
- net OUT_CHARGING_LIGHT: now also R2.2
- net OUT_ALTRN_CONTROL: now reaches BRD1.A14 (HS4)
- net OUT_ALTRN_CONTROL: now also R3.2
Other:
- note removed: "ETB Relay???"
- moved on the sheet: P56, P57

Commit message: #17, #18, #14, #13
Parts:
- added D2: D_Schottky, Diode_SMD:D_SMA, symbol Device:D_Schottky
- added D3: DNP, Diode_SMD:D_SMA, symbol Device:D_Schottky
- added J4: XH-10AW, Connector_JST:JST_XH_S10B-XH-A_1x10_P2.50mm_Horizontal, symbol Connector_Generic:Conn_01x10
- added R4: Jumper-Pad-Pad, hellen-one-common:PAD-0805-PAD, symbol hellen-one-common:Jumper-Pad-Pad
- J2: footprint Connector_Molex:Molex_SPOX_5267-10A_1x10_P2.50mm_Vertical -> Connector_JST:JST_XH_B10B-XH-A_1x10_P2.50mm_Vertical; MyComment (none) -> DNP; now left out of the parts list
Connections:
- net 12V_MR: now also J2.1 (Pin_1), J2.2 (Pin_2), D2.1 (K), D3.1 (K), J4.1 (Pin_1), J4.2 (Pin_2); no longer J2.10 (Pin_10), J2.9 (Pin_9)
- net GND: now also J2.10 (Pin_10), J2.9 (Pin_9), J4.10 (Pin_10), J4.9 (Pin_9); no longer J2.1 (Pin_1), J2.2 (Pin_2)
- net OUT_IAC: now also R4.2; no longer J1.A12
- net OUT_VTC: now also D2.2 (A)
- net OUT_VTS: now also D3.2 (A)
- net WBO_H-: now also J2.7 (Pin_7), J2.8 (Pin_8), J4.7 (Pin_7), J4.8 (Pin_8); no longer J2.3 (Pin_3), J2.4 (Pin_4)
- net WBO_Ip: now also J2.5 (Pin_5), J4.5 (Pin_5); no longer J2.6 (Pin_6)
- net WBO_R_Trim: now also J2.6 (Pin_6), J4.6 (Pin_6); no longer J2.5 (Pin_5)
- net WBO_Vs: now also J2.3 (Pin_3), J4.3 (Pin_3); no longer J2.8 (Pin_8)
- net WBO_Vs/Ip: now also J2.4 (Pin_4), J4.4 (Pin_4); no longer J2.7 (Pin_7)
- new net: J1.A12, R4.1
Other:
- moved on the sheet: J2
Changed lines of the file:
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@@
   (junction (at 104.14 392.43) (diameter 0) (color 0 0 0 0))
   (junction (at 104.14 398.78) (diameter 0) (color 0 0 0 0))
+  (junction (at 106.68 24.13) (diameter 0) (color 0 0 0 0))
   (junction (at 106.68 26.67) (diameter 0) (color 0 0 0 0))
+  (junction (at 106.68 29.21) (diameter 0) (color 0 0 0 0))
   (junction (at 106.68 31.75) (diameter 0) (color 0 0 0 0))
+  (junction (at 106.68 34.29) (diameter 0) (color 0 0 0 0))
+  (junction (at 106.68 36.83) (diameter 0) (color 0 0 0 0))
+  (junction (at 106.68 39.37) (diameter 0) (color 0 0 0 0))
+  (junction (at 106.68 41.91) (diameter 0) (color 0 0 0 0))
+  (junction (at 106.68 44.45) (diameter 0) (color 0 0 0 0))
+  (junction (at 106.68 46.99) (diameter 0) (color 0 0 0 0))
   (junction (at 119.38 373.38) (diameter 0) (color 0 0 0 0))
   (junction (at 119.38 379.73) (diameter 0) (color 0 0 0 0))
@@
     (stroke (width 0) (type solid) (color 0 0 0 0))
   )
-  (wire (pts (xy 36.83 46.99) (xy 71.12 46.99))
-    (stroke (width 0) (type solid) (color 0 0 0 0))
-  )
   (wire (pts (xy 36.83 49.53) (xy 71.12 49.53))
     (stroke (width 0) (type solid) (color 0 0 0 0))
@@
     (stroke (width 0) (type solid) (color 0 0 0 0))
   )
+  (wire (pts (xy 46.99 46.99) (xy 71.12 46.99))
+    (stroke (width 0) (type solid) (color 0 0 0 0))
+  )
   (wire (pts (xy 46.99 128.27) (xy 71.12 128.27))
     (stroke (width 0) (type solid) (color 0 0 0 0))
@@
     (stroke (width 0) (type default) (color 0 0 0 0))
   )
+  (wire (pts (xy 96.52 24.13) (xy 106.68 24.13))
+    (stroke (width 0) (type default) (color 0 0 0 0))
+  )
+  (wire (pts (xy 96.52 26.67) (xy 106.68 26.67))
+    (stroke (width 0) (type default) (color 0 0 0 0))
+  )
+  (wire (pts (xy 96.52 29.21) (xy 106.68 29.21))
+    (stroke (width 0) (type default) (color 0 0 0 0))
+  )
+  (wire (pts (xy 96.52 31.75) (xy 106.68 31.75))
+    (stroke (width 0) (type default) (color 0 0 0 0))
+  )
+  (wire (pts (xy 96.52 34.29) (xy 106.68 34.29))
+    (stroke (width 0) (type default) (color 0 0 0 0))
+  )
+  (wire (pts (xy 96.52 36.83) (xy 106.68 36.83))
+    (stroke (width 0) (type default) (color 0 0 0 0))
+  )
+  (wire (pts (xy 96.52 39.37) (xy 106.68 39.37))
+    (stroke (width 0) (type default) (color 0 0 0 0))
+  )
+  (wire (pts (xy 96.52 41.91) (xy 106.68 41.91))
+    (stroke (width 0) (type default) (color 0 0 0 0))
+  )
+  (wire (pts (xy 96.52 44.45) (xy 106.68 44.45))
+    (stroke (width 0) (type default) (color 0 0 0 0))
+  )
+  (wire (pts (xy 96.52 46.99) (xy 106.68 46.99))
+    (stroke (width 0) (type default) (color 0 0 0 0))
+  )
   (wire (pts (xy 100.33 373.38) (xy 104.14 373.38))
     (stroke (width 0) (type default) (color 0 0 0 0))
@@
     (effects (font (size 1.27 1.27)) (justify right bottom))
   )
+  (label "12V_MR" (at 78.74 105.41 0)
+    (effects (font (size 1.27 1.27)) (justify left bottom))
+  )
+  (label "12V_MR" (at 78.74 118.11 0)
+    (effects (font (size 1.27 1.27)) (justify left bottom))
+  )
   (label "12V_MR" (at 78.74 140.97 0)
     (effects (font (size 1.27 1.27)) (justify left bottom))
@@
     (pin "1")
   )
+  (symbol (lib_id "Device:D_Schottky") (at 74.93 105.41 180) (unit 1)
+    (in_bom yes) (on_board yes)
+    (property "Reference" "D2" (id 0) (at 74.93 99.9236 0))
+    (property "Value" "D_Schottky" (id 1) (at 74.93 102.235 0))
+    (property "Footprint" "Diode_SMD:D_SMA" (id 2) (at 74.93 105.41 0)
+      (effects (font (size 1.27 1.27)) hide)
+    )
+    (property "Datasheet" "~" (id 3) (at 74.93 105.41 0)
+      (effects (font (size 1.27 1.27)) hide)
+    )
+    (property "LCSC" "C8678" (id 4) (at 74.93 105.41 0)
+      (effects (font (size 1.27 1.27)) hide)
+    )
+    (property "LCSC_ext" "0" (id 5) (at 74.93 105.41 0)
+      (effects (font (size 1.27 1.27)) hide)
+    )
+    (pin "1")
+    (pin "2")
+  )
+  (symbol (lib_id "Device:D_Schottky") (at 74.93 118.11 180) (unit 1)
+    (in_bom yes) (on_board yes)
+    (property "Reference" "D3" (id 0) (at 74.93 112.6236 0))
+    (property "Value" "DNP" (id 1) (at 74.93 114.935 0))
+    (property "Footprint" "Diode_SMD:D_SMA" (id 2) (at 74.93 118.11 0)
+      (effects (font (size 1.27 1.27)) hide)
+    )
+    (property "Datasheet" "~" (id 3) (at 74.93 118.11 0)
+      (effects (font (size 1.27 1.27)) hide)
+    )
+    (property "LCSC_ext" "" (id 5) (at 74.93 118.11 0)
+      (effects (font (size 1.27 1.27)) hide)
+    )
+    (pin "1")
+    (pin "2")
+  )
   (symbol (lib_id "Device:D_Schottky") (at 74.93 140.97 180) (unit 1)
     (in_bom yes) (on_board yes)
@@
     (pin "2")
   )
+  (symbol (lib_id "hellen-one-common:Jumper-Pad-Pad") (at 41.91 46.99 0) (unit 1)
+    (in_bom yes) (on_board yes)
+    (property "Reference" "R4" (id 0) (at 46.99 45.8589 0)
+      (effects (font (size 1.016 1.016)))
+    )
+    (property "Value" "Jumper-Pad-Pad" (id 1) (at 41.91 48.768 0)
+      (effects (font (size 1.016 1.016)) hide)
+    )
+    (property "Footprint" "hellen-one-common:PAD-0805-PAD" (id 2) (at 41.91 50.8 0)
+      (effects (font (size 1.524 1.524)) hide)
+    )
+    (property "Datasheet" "" (id 3) (at 41.91 46.99 0)
+      (effects (font (size 1.524 1.524)) hide)
+    )
+    (property "LCSC" "C17477" (id 4) (at 41.91 50.8 0)
+      (effects (font (size 1.27 1.27)) hide)
+    )
+    (pin "1")
+    (pin "2")
+  )
   (symbol (lib_id "hellen-one-common:Jumper-Pad-Pad") (at 41.91 128.27 0) (unit 1)
     (in_bom yes) (on_board yes)
@@
     (pin "6")
   )
-  (symbol (lib_id "Connector_Generic:Conn_01x10") (at 101.6 34.29 0) (mirror y) (unit 1)
+  (symbol (lib_id "Connector_Generic:Conn_01x10") (at 91.44 36.83 180) (unit 1)
     (in_bom yes) (on_board yes) (fields_autoplaced)
+    (property "Reference" "J4" (id 0) (at 93.2815 18.8934 0))
+    (property "Value" "XH-10AW" (id 1) (at 93.2815 21.6685 0))
+    (property "Footprint" "Connector_JST:JST_XH_S10B-XH-A_1x10_P2.50mm_Horizontal" (id 2) (at 91.44 36.83 0)
+      (effects (font (size 1.27 1.27)) hide)
+    )
+    (property "Datasheet" "~" (id 3) (at 91.44 36.83 0)
+      (effects (font (size 1.27 1.27)) hide)
+    )
+    (property "LCSC" "C14652" (id 4) (at 91.44 36.83 0)
+      (effects (font (size 1.27 1.27)) hide)
+    )
+    (pin "1")
+    (pin "10")
+    (pin "2")
+    (pin "3")
+    (pin "4")
+    (pin "5")
+    (pin "6")
+    (pin "7")
+    (pin "8")
+    (pin "9")
+  )
+  (symbol (lib_id "Connector_Generic:Conn_01x10") (at 101.6 36.83 180) (unit 1)
+    (in_bom no) (on_board no)
     (property "Reference" "J2" (id 0) (at 103.4415 18.8934 0))
     (property "Value" "XH-10A" (id 1) (at 103.4415 21.6685 0))
-    (property "Footprint" "Connector_Molex:Molex_SPOX_5267-10A_1x10_P2.50mm_Vertical" (id 2) (at 101.6 34.29 0)
+    (property "Footprint" "Connector_JST:JST_XH_B10B-XH-A_1x10_P2.50mm_Vertical" (id 2) (at 101.6 36.83 0)
       (effects (font (size 1.27 1.27)) hide)
     )
-    (property "Datasheet" "~" (id 3) (at 101.6 34.29 0)
+    (property "Datasheet" "~" (id 3) (at 101.6 36.83 0)
       (effects (font (size 1.27 1.27)) hide)
     )
-    (property "LCSC" "C8885" (id 4) (at 101.6 34.29 0)
+    (property "LCSC" "C8885" (id 4) (at 101.6 36.83 0)
       (effects (font (size 1.27 1.27)) hide)
     )
+    (property "MyComment" "DNP" (id 5) (at 101.6 49.53 0))
     (pin "1")
     (pin "10")
@@
       (reference "D1") (unit 1) (value "D_Schottky") (footprint "Diode_SMD:D_SMA")
     )
+    (path "/6ab2b11f-ffcf-4597-a6e5-7a79f4782a77"
+      (reference "D2") (unit 1) (value "D_Schottky") (footprint "Diode_SMD:D_SMA")
+    )
+    (path "/4f201856-a058-412d-a76d-0c18de3afaf2"
+      (reference "D3") (unit 1) (value "DNP") (footprint "Diode_SMD:D_SMA")
+    )
     (path "/526071ab-b3d5-46b5-8fed-90eccd02a916"
       (reference "F1") (unit 1) (value "Fuse-Pad-Pad") (footprint "hellen-one-common:PAD-1206-PAD")
@@
     )
     (path "/1383430e-0b76-4a46-a167-f386c716d501"
-      (reference "J2") (unit 1) (value "XH-10A") (footprint "Connector_Molex:Molex_SPOX_5267-10A_1x10_P2.50mm_Vertical")
+      (reference "J2") (unit 1) (value "XH-10A") (footprint "Connector_JST:JST_XH_B10B-XH-A_1x10_P2.50mm_Vertical")
     )
     (path "/398f8f70-e91c-4da2-a829-819a6f9d0c83"
       (reference "J3") (unit 1) (value "Conn_01x06") (footprint "Connector_PinHeader_2.54mm:PinHeader_1x06_P2.54mm_Vertical")
     )
+    (path "/a4dd082f-21d1-49da-ab0f-42e564f3dbe1"
+      (reference "J4") (unit 1) (value "XH-10AW") (footprint "Connector_JST:JST_XH_S10B-XH-A_1x10_P2.50mm_Horizontal")
+    )
     (path "/fdce6d33-fe0a-477b-8253-68869a163636"
       (reference "J7") (unit 1) (value "Conn_01x01") (footprint "MountingHole:MountingHole_4.5mm")
@@
       (reference "R3") (unit 1) (value "Jumper-Pad-Pad") (footprint "hellen-one-common:PAD-0805-PAD")
     )
+    (path "/1b1d0c0f-875d-480b-89bb-24ea6bdac404"
+      (reference "R4") (unit 1) (value "Jumper-Pad-Pad") (footprint "hellen-one-common:PAD-0805-PAD")
+    )
     (path "/56d42875-db96-4dcd-87bf-57d53391facd"
